File: electronics/picr_1_9tdi.kicad_sch (KiCad schematic)
At the start: 73 parts, among them J1 Conn_01x03_Pin, J2 10118193-0001LF, J3 Conn_01x02_Socket, J4 Conn_01x02_Socket, J5 Conn_01x02_Socket, J6 Conn_01x02_Socket, J7 Conn_01x02_Socket, J9 Conn_01x02_Socket, Q1 BSC026N08NS5, U1 PDRV8243SDGQQ1, U10 NCP718BSN500T1G, U11 PDRV8243SDGQQ1, U12 PDRV8243SDGQQ1, U13 215079-4, U2 STM32G441KBT6, U3 CM1223-02SO, U4 MIC5504-3.3YM5, U5 NCP718BSN500T1G, U6 215079-4, U7 215079-4, U8 215079-4, U9 20021121-00010T4LF

Commit message: Schem rev2
Parts:
- removed C1: 10u, Library:C_1206_3216Metric_Pad1.33x1.80mm_HandSolder, symbol Library:C
- removed C4, C5, C6, C7: 100n, Library:C_1206_3216Metric_Pad1.33x1.80mm_HandSolder, symbol Library:C
- removed R1: 10K, Library:R_0201_0603Metric_Pad0.64x0.40mm_HandSolder, symbol Library:R
- removed U2: STM32G441KBT6, Library:LQFP-32_7x7mm_P0.8mm, symbol Library:STM32G441KBTx
- added C19: 10u, Capacitor_SMD:C_0805_2012Metric_Pad1.18x1.45mm_HandSolder, symbol Library:C
- added C20, C22, C23, C25: 100n, Capacitor_SMD:C_0603_1608Metric_Pad1.08x0.95mm_HandSolder, symbol Library:C
- added C30, C31: 0.1u, Capacitor_SMD:C_0603_1608Metric_Pad1.08x0.95mm_HandSolder, symbol Library:C
- added J9: Conn_01x03_Pin, Connector_PinHeader_2.54mm:PinHeader_1x03_P2.54mm_Vertical, symbol Library:Conn_01x03_Pin
- added R14: 10K, Resistor_SMD:R_0603_1608Metric_Pad0.98x0.95mm_HandSolder, symbol Library:R
- added U16: MAX12930EASA+, Library:SOIC-8_L4.9-W3.9-P1.27-LS6.0-BL, symbol Library:MAX12930EASA+
- added U8: STM32G441KBT6, Library:LQFP-32_7x7mm_P0.8mm, symbol Library:KBT6
- C1: renamed from C27; footprint Library:C_1206_3216Metric_Pad1.33x1.80mm_HandSolder -> Capacitor_SMD:C_0805_2012Metric_Pad1.18x1.45mm_HandSolder
- C10: renamed from C16; footprint Library:C_1206_3216Metric_Pad1.33x1.80mm_HandSolder -> Capacitor_SMD:C_0805_2012Metric_Pad1.18x1.45mm_HandSolder
- C11: renamed from C8; footprint Library:C_1206_3216Metric_Pad1.33x1.80mm_HandSolder -> Capacitor_SMD:C_0603_1608Metric_Pad1.08x0.95mm_HandSolder
- C12: renamed from C2; footprint Library:C_1206_3216Metric_Pad1.33x1.80mm_HandSolder -> Capacitor_SMD:C_0603_1608Metric_Pad1.08x0.95mm_HandSolder
- C13: renamed from C17; footprint Library:C_1206_3216Metric_Pad1.33x1.80mm_HandSolder -> Capacitor_SMD:C_0805_2012Metric_Pad1.18x1.45mm_HandSolder
- C14: renamed from C18; footprint Library:C_1206_3216Metric_Pad1.33x1.80mm_HandSolder -> Capacitor_SMD:C_0805_2012Metric_Pad1.18x1.45mm_HandSolder
- C15: renamed from C3; footprint Library:C_1206_3216Metric_Pad1.33x1.80mm_HandSolder -> Capacitor_SMD:C_0603_1608Metric_Pad1.08x0.95mm_HandSolder
- C16: renamed from C9; footprint Library:C_1206_3216Metric_Pad1.33x1.80mm_HandSolder -> Capacitor_SMD:C_0603_1608Metric_Pad1.08x0.95mm_HandSolder
- C17: renamed from C19; footprint Library:C_1206_3216Metric_Pad1.33x1.80mm_HandSolder -> Capacitor_SMD:C_0603_1608Metric_Pad1.08x0.95mm_HandSolder
- C18: renamed from C20; footprint Library:C_1206_3216Metric_Pad1.33x1.80mm_HandSolder -> Capacitor_SMD:C_0603_1608Metric_Pad1.08x0.95mm_HandSolder
- C2: renamed from C26; footprint Library:C_1206_3216Metric_Pad1.33x1.80mm_HandSolder -> Capacitor_SMD:C_0805_2012Metric_Pad1.18x1.45mm_HandSolder
- C21: footprint Library:C_1206_3216Metric_Pad1.33x1.80mm_HandSolder -> Capacitor_SMD:C_0805_2012Metric_Pad1.18x1.45mm_HandSolder
- C24: renamed from C22; footprint Library:C_1206_3216Metric_Pad1.33x1.80mm_HandSolder -> Capacitor_SMD:C_0805_2012Metric_Pad1.18x1.45mm_HandSolder
- C26: renamed from C23; footprint Library:C_1206_3216Metric_Pad1.33x1.80mm_HandSolder -> Capacitor_SMD:C_0805_2012Metric_Pad1.18x1.45mm_HandSolder
- C27: renamed from C25; footprint Library:C_1206_3216Metric_Pad1.33x1.80mm_HandSolder -> Capacitor_SMD:C_0805_2012Metric_Pad1.18x1.45mm_HandSolder
- C28, C29: footprint Library:C_1206_3216Metric_Pad1.33x1.80mm_HandSolder -> Capacitor_SMD:C_0603_1608Metric_Pad1.08x0.95mm_HandSolder
- C3: renamed from C14; footprint Library:C_1206_3216Metric_Pad1.33x1.80mm_HandSolder -> Capacitor_SMD:C_0805_2012Metric_Pad1.18x1.45mm_HandSolder
- C4: renamed from C12; footprint Library:C_1206_3216Metric_Pad1.33x1.80mm_HandSolder -> Capacitor_SMD:C_0805_2012Metric_Pad1.18x1.45mm_HandSolder
- C5: renamed from C15; footprint Library:C_1206_3216Metric_Pad1.33x1.80mm_HandSolder -> Capacitor_SMD:C_0603_1608Metric_Pad1.08x0.95mm_HandSolder
- C6: renamed from C10; footprint Library:C_1206_3216Metric_Pad1.33x1.80mm_HandSolder -> Capacitor_SMD:C_0603_1608Metric_Pad1.08x0.95mm_HandSolder
- C7: renamed from C24; footprint Library:C_1206_3216Metric_Pad1.33x1.80mm_HandSolder -> Capacitor_SMD:C_0603_1608Metric_Pad1.08x0.95mm_HandSolder
- C8: renamed from C11; footprint Library:C_1206_3216Metric_Pad1.33x1.80mm_HandSolder -> Capacitor_SMD:C_0603_1608Metric_Pad1.08x0.95mm_HandSolder
- C9: renamed from C13; footprint Library:C_1206_3216Metric_Pad1.33x1.80mm_HandSolder -> Capacitor_SMD:C_0805_2012Metric_Pad1.18x1.45mm_HandSolder
- R1: renamed from R6; footprint Library:R_0201_0603Metric_Pad0.64x0.40mm_HandSolder -> Resistor_SMD:R_0603_1608Metric_Pad0.98x0.95mm_HandSolder
- R10: renamed from R13; footprint Library:R_0201_0603Metric_Pad0.64x0.40mm_HandSolder -> Resistor_SMD:R_0603_1608Metric_Pad0.98x0.95mm_HandSolder
- R11: renamed from R5; footprint Library:R_0201_0603Metric_Pad0.64x0.40mm_HandSolder -> Resistor_SMD:R_0603_1608Metric_Pad0.98x0.95mm_HandSolder
- R12: renamed from R15; value 500R -> 2K7; footprint Library:R_0201_0603Metric_Pad0.64x0.40mm_HandSolder -> Resistor_SMD:R_0603_1608Metric_Pad0.98x0.95mm_HandSolder
- R13: renamed from R16; value 2K -> 100K; footprint Library:R_0201_0603Metric_Pad0.64x0.40mm_HandSolder -> Resistor_SMD:R_0603_1608Metric_Pad0.98x0.95mm_HandSolder
- R15: renamed from R17; footprint Library:R_0201_0603Metric_Pad0.64x0.40mm_HandSolder -> Resistor_SMD:R_0603_1608Metric_Pad0.98x0.95mm_HandSolder
- R16: renamed from R18; footprint Library:R_0201_0603Metric_Pad0.64x0.40mm_HandSolder -> Resistor_SMD:R_0603_1608Metric_Pad0.98x0.95mm_HandSolder
- R17: renamed from R19; value 500R -> 2K7; footprint Library:R_0201_0603Metric_Pad0.64x0.40mm_HandSolder -> Resistor_SMD:R_0603_1608Metric_Pad0.98x0.95mm_HandSolder
- R18: renamed from R8; footprint Library:R_0201_0603Metric_Pad0.64x0.40mm_HandSolder -> Resistor_SMD:R_0603_1608Metric_Pad0.98x0.95mm_HandSolder
- R19: renamed from R7; footprint Library:R_0201_0603Metric_Pad0.64x0.40mm_HandSolder -> Resistor_SMD:R_0603_1608Metric_Pad0.98x0.95mm_HandSolder
- R2: value 2K -> 100K; footprint Library:R_0201_0603Metric_Pad0.64x0.40mm_HandSolder -> Resistor_SMD:R_0603_1608Metric_Pad0.98x0.95mm_HandSolder
- R3: renamed from R14; footprint Library:R_0201_0603Metric_Pad0.64x0.40mm_HandSolder -> Resistor_SMD:R_0603_1608Metric_Pad0.98x0.95mm_HandSolder
- R4: renamed from R12; footprint Library:R_0201_0603Metric_Pad0.64x0.40mm_HandSolder -> Resistor_SMD:R_0603_1608Metric_Pad0.98x0.95mm_HandSolder
- R5: renamed from R9; value 500R -> 2K7; footprint Library:R_0201_0603Metric_Pad0.64x0.40mm_HandSolder -> Resistor_SMD:R_0603_1608Metric_Pad0.98x0.95mm_HandSolder
- R6: renamed from R3; footprint Library:R_0201_0603Metric_Pad0.64x0.40mm_HandSolder -> Resistor_SMD:R_0603_1608Metric_Pad0.98x0.95mm_HandSolder
- R7: renamed from R4; footprint Library:R_0201_0603Metric_Pad0.64x0.40mm_HandSolder -> Resistor_SMD:R_0603_1608Metric_Pad0.98x0.95mm_HandSolder
- R8: renamed from R10; value 2K -> 100K; footprint Library:R_0201_0603Metric_Pad0.64x0.40mm_HandSolder -> Resistor_SMD:R_0603_1608Metric_Pad0.98x0.95mm_HandSolder
- R9: renamed from R11; footprint Library:R_0201_0603Metric_Pad0.64x0.40mm_HandSolder -> Resistor_SMD:R_0603_1608Metric_Pad0.98x0.95mm_HandSolder
- renumbered D3 to D1, J2 to J1, J6 to J2, J9 to J3, J1 to J4, J7 to J5, J5 to J6, J3 to J7, J4 to J8, U13 to U10, U6 to U11, U7 to U12, U16 to U13, U17 to U14, U8 to U15, U3 to U2, U5 to U3, U11 to U4, U4 to U5, U10 to U6, U12 to U7
Connections:
- net +3.3V: now also C19.1, C20.1, C22.1, C25.1, C30.1, U16.1 (VDDA), U8.1 (VDD), U8.15 (VDDA), U8.17 (VDD)
- net D+: now also U8.22 (PA12)
- net D-: now also U8.21 (PA11)
- net E_M1_A: now also U8.5 (PA0)
- net E_M1_B: now also U8.6 (PA1)
- net E_M2_A: now also U8.9 (PA4)
- net E_M2_B: now also U8.11 (PA6)
- net E_M3_A: now also U8.29 (PB6)
- net E_M3_B: now also U8.30 (PB7)
- net IR_RX: now also U8.3 (PF1)
- net M1_DIR_I: now also U8.7 (PA2)
- net M2_DIR_I: now also U8.8 (PA3)
- net M3_DIR_I: now also U8.10 (PA5)
- net M_NSLEEP_I: now also U8.12 (PA7)
- net NRST: now also C23.1, U8.4 (PG10)
- net PWM_M1_I: now also U8.18 (PA8)
- net PWM_M2_I: now also U8.19 (PA9)
- net PWM_M3_I: now also U8.20 (PA10)
- net PWM_TH_I: now also U8.25 (PA15)
- net SWCLK: now also U8.24 (PA14)
- net SWDIO: now also U8.23 (PA13)
- net V_SERVO: now also J9.2 (Pin_2)
- net +5V renamed 5V_MOT
- net 5V_MOT: now also C31.1, U16.8 (VDDB); no longer C12.1, J1.1 (VUSB), R6.1, R7.1, U2.5 (VP), U5.1 (VIN)
- net GND1 renamed GND_MCU
- net GND_MCU: now also C19.2, C20.2, C22.2, C23.2, C25.2, C30.2, R14.1, U16.4 (GNDA), U8.14 (VSSA), U8.16 (VSS), U8.32 (VSS); no longer C11.2, C16.2, C6.2, C8.2, D1.1 (K), J2.2 (Pin_2), J4.3 (Pin_3), Q1.4 (G), R1.2, U10.1 (GND), U11.1 (GND), U12.1 (GND), U15.3 (GND), U3.2 (GND), U6.2 (GND)
- net GND2 renamed GND_MOT
- net GND_MOT: now also C11.2, C16.2, C6.2, C8.2, D1.1 (K), J2.2 (Pin_2), J4.3 (Pin_3), Q1.4 (G), R1.2, U10.1 (GND), U11.1 (GND), U12.1 (GND), U15.3 (GND), U3.2 (GND), U6.2 (GND), C31.2, J9.3 (Pin_3), U16.5 (GNDB)
- net PWM_SER renamed PWM_GRB_O
- net PWM_GRB_O: now also U16.7 (OUT1)
- new net: R14.2, U8.31 (PB8)
- new net PWM_ANG_I: U16.3 (IN2), U8.28 (PB5)
- new net PWM_ANG_O: J9.1 (Pin_1), U16.6 (OUT2)
- new net PWM_GRB_I: U16.2 (IN1), U8.27 (PB4)
- new net VUSB: C12.1, J1.1 (VUSB), R6.1, R7.1, U2.5 (VP), U5.1 (VIN)
Other:
- note added: "ANGLE SERVO"
- note added: "GRABBER SERVO"
- note added: "Itrip lvl 5"
- note added: "VUSB -> 3V3"
- note removed: "5V -> 3V3"
- note removed: "SERVO"
- moved on the sheet: J4, J5, R18, R19, R6, U13, U14, U15

Commit message: .
Connections:
- net 5V_MOT: no longer R11.1
- net GND_MCU: now also D1.1 (K), U10.1 (GND), U11.1 (GND), U12.1 (GND)
- net GND_MOT: no longer D1.1 (K), U10.1 (GND), U11.1 (GND), U12.1 (GND)
- net VUSB: now also R11.1
Other:
- moved on the sheet: C30, C31, J5, J9, U15, U16

Commit message: .
Parts:
- removed U6: NCP718BSN500T1G, Library:SOT-23-5, symbol Library:NCP718xSN500
- added C32, C33: 100n, Capacitor_SMD:C_0603_1608Metric_Pad1.08x0.95mm_HandSolder, symbol Library:C
- added C34: 10u, Capacitor_SMD:C_0603_1608Metric_Pad1.08x0.95mm_HandSolder, symbol Library:C
- added L1: TBD, symbol Device:L
- added R20: TBD, Resistor_SMD:R_0603_1608Metric_Pad0.98x0.95mm_HandSolder, symbol Library:R
- added R21: 52K3, symbol Library:R
- added R22: 10K, Resistor_SMD:R_0603_1608Metric_Pad0.98x0.95mm_HandSolder, symbol Library:R
- added U6: TPS62933, Package_TO_SOT_SMD:SOT-583-8, symbol Regulator_Switching:TPS62933
- C11: value 1u -> 10u; footprint Capacitor_SMD:C_0603_1608Metric_Pad1.08x0.95mm_HandSolder -> Capacitor_SMD:C_0805_2012Metric_Pad1.18x1.45mm_HandSolder
- C16: value 1u -> 100n
Connections:
- net GND_MOT: now also C32.2, C34.2, R20.2, R22.2, U6.4 (GND)
- net VBAT: now also C16.1, U6.3 (VIN)
- net V_SERVO: now also C34.1, L1.2, R21.1; no longer C16.1
- new net: R21.2, R22.1, U6.8 (FB)
- new net: C33.2, L1.1, U6.5 (SW)
- new net: C33.1, U6.6 (BST)
- new net: C32.1, U6.7 (SS)
- new net: R20.1, U6.1 (RT)
Other:
- note added: "Fsw 2200 KHz"
- note added: "VBAT -> 5V SERVO"
- note removed: "VBAT -> SERVO 5V"
- moved on the sheet: C12, C15, C6, C8, D1, R11, U15, U3, U5

Commit message: .
Parts:
- removed J1: 10118193-0001LF, Library:USB_Micro-B_Amphenol_10118193-0001LF_Horizontal, symbol Library:10118193-0001LF
- removed Q1: BSC026N08NS5, Library:BUK6Y10-30PX, symbol Library:BSC026N08NS5
- removed R1: 100K, Resistor_SMD:R_0603_1608Metric_Pad0.98x0.95mm_HandSolder, symbol Library:R
- removed U15: 215079-4, Library:TE_Micro-MaTch_215079-4_2x02_P1.27mm_Vertical, symbol Library:215079-4_PWM
- removed U6: TPS62933, Package_TO_SOT_SMD:SOT-583-8, symbol Regulator_Switching:TPS62933
- added J1: USB_B_Micro_copy, symbol Library:USB_B_Micro_copy
- added Q1: AON6411_copy, Package_DFN_QFN:AO_DFN-8-1EP_5.55x5.2mm_P1.27mm_EP4.12x4.6mm, symbol Library:AON6411_copy
- added U16: ~, Library:TE_Micro-MaTch_215079-4_2x02_P1.27mm_Vertical, symbol Library:215079-4_PWM
- added U17: TPS62933_copy, Package_TO_SOT_SMD:SOT-583-8, symbol Library:TPS62933_copy
- L1: symbol Device:L -> Library:L
- R12: renamed from R21; footprint (none) -> Resistor_SMD:R_0603_1608Metric_Pad0.98x0.95mm_HandSolder
- U10: symbol Library:215079-4 -> Library:215079-4_1
- U11: symbol Library:215079-4 -> Library:215079-4_2
- U13, U14: footprint Library:SI8640AB-B-IS1 -> ProLib_pcs_2025-09-23 (1):SOIC-16_L9.9-W3.9-P1.27-LS5.9-BL
- U3: footprint Library:SOT-23-5 -> Package_TO_SOT_SMD:SOT-23-5
- U4: renamed from U5; footprint Library:SOT-23-5 -> Package_TO_SOT_SMD:SOT-23-5
- U9: footprint Library:HDR-SMD_10P-P1.27-V-M-R2-C5-S1.27-LS5.5 -> ProLib_pcs_2025-09-19 (1):HDR-SMD_10P-P1.27-V-M-R2-C5-S1.27-LS5.5
- renumbered C15 to C10, C9 to C12, C16 to C13, C10 to C14, C32 to C15, C13 to C16, C14 to C17, C33 to C18, C17 to C19, C34 to C20, C18 to C21, C19 to C22, C20 to C23, C21 to C24, C22 to C25, C23 to C26, C24 to C27, C25 to C28, C26 to C29, C27 to C30, C28 to C31, C29 to C32, C30 to C33, C31 to C34, C6 to C5, C5 to C6, C12 to C7, C7 to C8, C8 to C9, J9 to J6, J6 to J7, J7 to J8, J8 to J9, R2 to R1, R22 to R13, R12 to R14, R13 to R15, R14 to R16, R15 to R17, R16 to R18, R17 to R19, R3 to R2, R18 to R20, R19 to R21, R4 to R3, R5 to R4, R6 to R5, R7 to R6, R8 to R7, R20 to R8, U16 to U15, U4 to U6
Connections:
- net D+: now also J1.3 (D+)
- net D-: now also J1.2 (D-)
- net GND_MCU: now also J1.5 (GND), J1.6 (Shield)
- net GND_MOT: now also Q1.4 (G), U16.1, U17.4 (GND)
- net PWM_TH_O: now also U16.2
- net VBAT: now also Q1.5 (D), U17.3 (VIN)
- net VBAT_IN: now also Q1.1 (S), Q1.2 (S), Q1.3 (S)
- net VUSB: now also J1.1 (VBUS)
- net at R12.2, R13.1: now also U17.8 (FB)
- net at C18.2, L1.1: now also U17.5 (SW)
- net at C18.1: now also U17.6 (BST)
- net at C15.1: now also U17.7 (SS)
- net at R8.1: now also U17.1 (RT)
Other:
- moved on the sheet: J5

Commit message: Schem rev3
Parts:
- added C33, C34, C35, C36: 0.1u, Capacitor_SMD:C_0603_1608Metric_Pad1.08x0.95mm_HandSolder, symbol Library:C
- J1: footprint (none) -> Library:USB_Micro-B_Amphenol_10118193-0001LF_Horizontal
- L1: value TBD -> 1.5u; footprint (none) -> Inductor_SMD:SRP4021HMCT-1R5M_custom
- Q1: footprint Package_DFN_QFN:AO_DFN-8-1EP_5.55x5.2mm_P1.27mm_EP4.12x4.6mm -> Library:BUK6Y10-30PX
- R8: value TBD -> 35K
- U13, U14: footprint ProLib_pcs_2025-09-23 (1):SOIC-16_L9.9-W3.9-P1.27-LS5.9-BL -> Library:SI8640AB-B-IS1
- U5: renamed from U17; value TPS62933_copy -> TPS62933
- U9: footprint ProLib_pcs_2025-09-19 (1):HDR-SMD_10P-P1.27-V-M-R2-C5-S1.27-LS5.5 -> Library:HDR-SMD_10P-P1.27-V-M-R2-C5-S1.27-LS5.5
- renumbered C33 to C37, C34 to C38
Connections:
- net +3.3V: now also C33.1, C34.1
- net 5V_MOT: now also C35.1, C36.1; no longer R20.1, R21.1
- net E_M2_A: now also U8.11 (PA6); no longer U8.9 (PA4)
- net E_M2_B: now also U8.9 (PA4); no longer U8.11 (PA6)
- net GND_MCU: now also C33.2, C34.2
- new net: C36.2, R21.1
- new net: C35.2, R20.1
Other:
- note added: "Fsw 600 KHz"
- note removed: "Fsw 2200 KHz"
- moved on the sheet: C37, C38, J5, R20, R21, U13, U14, U15, U16

Commit message: .
Parts:
- removed C36: 0.1u, Capacitor_SMD:C_0603_1608Metric_Pad1.08x0.95mm_HandSolder, symbol Library:C
- removed C5, C9: 1u, Capacitor_SMD:C_0603_1608Metric_Pad1.08x0.95mm_HandSolder, symbol Library:C
- removed J3: Conn_01x02_Socket, Library:SolderWirePad_1x02_SMD_3x4mm, symbol Library:Conn_01x02_Socket
- removed R6: 100K, Resistor_SMD:R_0603_1608Metric_Pad0.98x0.95mm_HandSolder, symbol Library:R
- removed U3: NCP718BSN500T1G, Package_TO_SOT_SMD:SOT-23-5, symbol Library:NCP718xSN500
- added C12: 10u, Capacitor_SMD:C_0603_1608Metric_Pad1.08x0.95mm_HandSolder, symbol Library:C
- added C34: 0.1u, Capacitor_SMD:C_0603_1608Metric_Pad1.08x0.95mm_HandSolder, symbol Library:C
- added J3: Conn_01x03_Pin, Connector_PinHeader_2.54mm:PinHeader_1x03_P2.54mm_Vertical, symbol Library:Conn_01x03_Pin
- D1: footprint Library:LED_0201_0603Metric_Pad0.64x0.40mm_HandSolder -> LED_SMD:LED_0603_1608Metric_Pad1.05x0.95mm_HandSolder
- J2, J7, J8, J9: footprint Library:SolderWirePad_1x02_SMD_3x4mm -> Connector_Wire:SolderWirePad_1x02_SMD_3x4mm
- R12: renamed from R11; value 100R -> 4K7
- R4: renamed from R8; value 35K -> 10K
- R6: renamed from R5; value 100R -> 68R
- renumbered C18 to C10, C20 to C11, C12 to C13, C16 to C15, C7 to C16, C10 to C18, C21 to C20, C22 to C21, C23 to C22, C24 to C23, C25 to C24, C26 to C25, C27 to C26, C28 to C27, C29 to C28, C30 to C29, C31 to C30, C32 to C31, C34 to C32, C37 to C36, C38 to C37, C11 to C5, C13 to C6, C6 to C7, C15 to C8, C8 to C9, R9 to R10, R10 to R11, R14 to R13, R15 to R14, R16 to R15, R17 to R16, R18 to R17, R19 to R18, R20 to R19, R21 to R20, R4 to R5, R12 to R7, R13 to R8, R7 to R9, U11 to U10, U12 to U11, U13 to U12, U14 to U13, U15 to U14, U16 to U15, U5 to U3, U6 to U4, U4 to U5, U7 to U6, U8 to U7, U9 to U8, U10 to U9
Connections:
- net V_SERVO is gone; now on net 5V_MOT: C11.1, J4.2 (Pin_2), J6.2 (Pin_2), L1.2, R7.1
- net 5V_MOT: now also R19.1, R20.1, C12.1, C34.1
- net GND_MCU: now also J3.3 (Pin_3)
- net GND_MOT: now also C35.2, C12.2, C34.2
- net IR_RX: now also J3.2 (Pin_2)
- net VBAT: now also Q1.1 (S), Q1.2 (S), Q1.3 (S); no longer Q1.5 (D)
- net VBAT_IN: now also Q1.5 (D); no longer Q1.1 (S), Q1.2 (S), Q1.3 (S)
- net VUSB: now also J3.1 (Pin_1)
Other:
- note added: "Fsw ~1900 KHz"
- note added: "IR TX"
- note added: "RX (IS471FE)"
- note added: "TX (IR LED 3mm)"
- note added: "VBAT -> 5V"
- note removed: "Fsw 600 KHz"
- note removed: "IR RX/TX"
- note removed: "RX (IR DIODE)"
- note removed: "RX (IR DIODE, rev bias)"
- note removed: "TO MCU ADC"
- note removed: "VBAT -> 5V SERVO"
- note removed: "VBAT-> 5V"
- moved on the sheet: C10, C11, C16, C18, C5, C6, C8, L1, Q1, R4, R6, R7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

Commit message: .
Other:
- note added: "FROM IR RX (IS471FE)"
- note added: "TO IR TX (IR LED 3mm)"
- note added: "gpio_input"
- note removed: "RX (IS471FE)"
- note removed: "TX (IR LED 3mm)"
Changed lines of the file:
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@@
 		)
 	)
-	(text "TX (IR LED 3mm)"
+	(text "TO IR TX (IR LED 3mm)"
 		(exclude_from_sim no)
 		(at 480.314 333.756 0)
@@
 		)
 	)
+	(text "gpio_input"
+		(exclude_from_sim no)
+		(at 311.404 176.784 0)
+		(effects
+			(font
+				(size 1.27 1.27)
+			)
+		)
+	)
 	(text "GRABBER SERVO"
 		(exclude_from_sim no)
@@
 	(text "TX (IR LED)"
 		(exclude_from_sim no)
-		(at 146.812 139.954 0)
+		(at 144.526 138.684 0)
 		(effects
 			(font
@@
 		)
 	)
-	(text "RX (IS471FE)"
+	(text "FROM IR RX (IS471FE)"
 		(exclude_from_sim no)
-		(at 436.626 332.994 0)
+		(at 440.944 332.994 0)
 		(effects
 			(font
@@
 	(wire
 		(pts
-			(xy 436.88 342.9) (xy 436.88 349.25)
+			(xy 435.61 342.9) (xy 435.61 349.25)
 		)
 		(stroke
@@
 	(wire
 		(pts
+			(xy 435.61 342.9) (xy 436.88 342.9)
+		)
+		(stroke
+			(width 0)
+			(type default)
+		)
+	)
+	(wire
+		(pts
 			(xy 444.5 191.77) (xy 447.04 191.77)
 		)
@@
 	(wire
 		(pts
-			(xy 430.53 337.82) (xy 436.88 337.82)
+			(xy 425.45 337.82) (xy 436.88 337.82)
 		)
 		(stroke
@@
 	(wire
 		(pts
-			(xy 430.53 340.36) (xy 436.88 340.36)
+			(xy 425.45 340.36) (xy 436.88 340.36)
 		)
 		(stroke
@@
 	)
 	(label "VUSB"
-		(at 430.53 337.82 180)
+		(at 425.45 337.82 180)
 		(effects
 			(font
@@
 	)
 	(label "IR_RX"
-		(at 430.53 340.36 180)
+		(at 425.45 340.36 180)
 		(effects
 			(font
@@
 	(symbol
 		(lib_id "Library:GND")
-		(at 436.88 349.25 0)
+		(at 435.61 349.25 0)
 		(unit 1)
 		(exclude_from_sim no)
@@
 		(fields_autoplaced yes)
 		(property "Reference" "#PWR035"
-			(at 436.88 355.6 0)
+			(at 435.61 355.6 0)
 			(effects
 				(font
@@
 		)
 		(property "Value" "GND_MCU"
-			(at 436.88 354.33 0)
+			(at 435.61 354.33 0)
 			(effects
 				(font
@@
 		)
 		(property "Footprint" ""
-			(at 436.88 349.25 0)
+			(at 435.61 349.25 0)
 			(effects
 				(font
@@
 		)
 		(property "Datasheet" ""
-			(at 436.88 349.25 0)
+			(at 435.61 349.25 0)
 			(effects
 				(font
@@
 		)
 		(property "Description" "Power symbol creates a global label with name \"GND\" , ground"
-			(at 436.88 349.25 0)
+			(at 435.61 349.25 0)
 			(effects
 				(font

Commit message: .
Connections:
- net VUSB: no longer R12.1
- net MCU_LED: now reaches U7.26 (PB3)
- net MCU_LED: now also R12.1
Changed lines of the file:
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@@
+	(wire
+		(pts
+			(xy 321.31 185.42) (xy 326.39 185.42)
+		)
+		(stroke
+			(width 0)
+			(type default)
+		)
+	)
 	(wire
 		(pts
@@
 		)
 	)
-	(label "VUSB"
-		(at 191.77 139.7 180)
-		(effects
-			(font
-				(size 1.27 1.27)
-			)
-			(justify right bottom)
-		)
-	)
 	(label "E_M3_A"
 		(at 435.61 308.61 180)
@@
 		)
 	)
+	(label "MCU_LED"
+		(at 191.77 139.7 180)
+		(effects
+			(font
+				(size 1.27 1.27)
+			)
+			(justify right bottom)
+		)
+	)
 	(label "M_NSLEEP_O"
 		(at 57.15 316.23 180)
@@
 		(effects
 			(font
+				(size 1.27 1.27)
+			)
+			(justify right bottom)
+		)
+	)
+	(label "MCU_LED"
+		(at 321.31 185.42 180)
+		(effects
+			(font
