File: electronics/picr_1_9tdi.kicad_sch (KiCad schematic)
At the start: 84 parts, among them J1 USB_B_Micro_copy, J2 Conn_01x02_Socket, J3 Conn_01x03_Pin, J4 Conn_01x03_Pin, J5 Conn_01x02_Socket, J6 Conn_01x03_Pin, J7 Conn_01x02_Socket, J8 Conn_01x02_Socket, J9 Conn_01x02_Socket, Q1 AON6411_copy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

Commit message: .
Parts:
- removed J3: Conn_01x03_Pin, Connector_PinHeader_2.54mm:PinHeader_1x03_P2.54mm_Vertical, symbol Library:Conn_01x03_Pin
- added J3: Conn_01x04_Socket, Connector_PinHeader_2.54mm:PinHeader_1x04_P2.54mm_Vertical, symbol Library:Conn_01x04_Socket
- C10, C22, C24, C25, C27, C6, C8: value 100n -> 0.1u
- J1: value USB_B_Micro_copy -> 10118193-0001LF
- Q1: value AON6411_copy -> BUK6Y10-30PX
- U1, U4, U6: value PDRV8243SDGQQ1 -> DRV8243HQDGQRQ1
- U12, U13: value ~ -> SI8640AB-B-IS1
- U15: value ~ -> 215079-4
Connections:
- net GND_MCU: now also J3.3 (Pin_3)
- net IR_RX: now also J3.2 (Pin_2)
- net IR_TX: now also J3.4 (Pin_4)
- net VUSB: now also J3.1 (Pin_1)

Commit message: .
Parts:
- J2, J7, J8, J9: footprint Connector_Wire:SolderWirePad_1x02_SMD_3x4mm -> Library:SolderWirePad_1x02_SMD_3x4mm
- J3: footprint Connector_PinHeader_2.54mm:PinHeader_1x04_P2.54mm_Vertical -> Library:PinHeader_1x04_P2.54mm_Vertical
- J4, J6: footprint Connector_PinHeader_2.54mm:PinHeader_1x03_P2.54mm_Vertical -> Library:PinHeader_1x03_P2.54mm_Vertical
- L1: footprint Inductor_SMD:SRP4021HMCT-1R5M_custom -> Library:SRP4021HMCT-1R5M_custom
- U3: footprint Package_TO_SOT_SMD:SOT-583-8 -> Library:SOT-583-8
- U5: footprint Package_TO_SOT_SMD:SOT-23-5 -> Library:SOT-23-5
Changed lines of the file:
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@@
 			)
 		)
-		(property "Footprint" "Connector_PinHeader_2.54mm:PinHeader_1x03_P2.54mm_Vertical"
+		(property "Footprint" "Library:PinHeader_1x03_P2.54mm_Vertical"
 			(at 505.46 242.57 0)
 			(effects
@@
 			)
 		)
-		(property "Footprint" "Package_TO_SOT_SMD:SOT-23-5"
+		(property "Footprint" "Library:SOT-23-5"
 			(at 207.01 232.41 0)
 			(effects
@@
 			)
 		)
-		(property "Footprint" "Package_TO_SOT_SMD:SOT-583-8"
+		(property "Footprint" "Library:SOT-583-8"
 			(at 113.03 213.36 0)
 			(effects
@@
 			)
 		)
-		(property "Footprint" "Inductor_SMD:SRP4021HMCT-1R5M_custom"
+		(property "Footprint" "Library:SRP4021HMCT-1R5M_custom"
 			(at 132.08 187.96 0)
 			(effects
@@
 			)
 		)
-		(property "Footprint" "Connector_Wire:SolderWirePad_1x02_SMD_3x4mm"
+		(property "Footprint" "Library:SolderWirePad_1x02_SMD_3x4mm"
 			(at 542.29 337.82 0)
 			(effects
@@
 			)
 		)
-		(property "Footprint" "Connector_PinHeader_2.54mm:PinHeader_1x03_P2.54mm_Vertical"
+		(property "Footprint" "Library:PinHeader_1x03_P2.54mm_Vertical"
 			(at 450.85 241.3 0)
 			(effects
@@
 			)
 		)
-		(property "Footprint" "Connector_Wire:SolderWirePad_1x02_SMD_3x4mm"
+		(property "Footprint" "Library:SolderWirePad_1x02_SMD_3x4mm"
 			(at 35.56 193.04 0)
 			(effects
@@
 			)
 		)
-		(property "Footprint" "Connector_Wire:SolderWirePad_1x02_SMD_3x4mm"
+		(property "Footprint" "Library:SolderWirePad_1x02_SMD_3x4mm"
 			(at 543.56 290.83 0)
 			(effects
@@
 			)
 		)
-		(property "Footprint" "Connector_PinHeader_2.54mm:PinHeader_1x04_P2.54mm_Vertical"
+		(property "Footprint" "Library:PinHeader_1x04_P2.54mm_Vertical"
 			(at 447.04 340.36 0)
 			(effects
@@
 			)
 		)
-		(property "Footprint" "Connector_Wire:SolderWirePad_1x02_SMD_3x4mm"
+		(property "Footprint" "Library:SolderWirePad_1x02_SMD_3x4mm"
 			(at 544.83 313.69 0)
 			(effects

Commit message: .
Parts:
- J3: footprint Library:PinHeader_1x04_P2.54mm_Vertical -> Connector_PinHeader_2.54mm:PinHeader_1x04_P2.54mm_Vertical
- J4, J6: footprint Library:PinHeader_1x03_P2.54mm_Vertical -> Connector_PinHeader_2.54mm:PinHeader_1x03_P2.54mm_Vertical
Changed lines of the file:
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@@
 			)
 		)
-		(property "Footprint" "Library:PinHeader_1x03_P2.54mm_Vertical"
+		(property "Footprint" "Connector_PinHeader_2.54mm:PinHeader_1x03_P2.54mm_Vertical"
 			(at 505.46 242.57 0)
 			(effects
@@
 			)
 		)
-		(property "Footprint" "Library:PinHeader_1x03_P2.54mm_Vertical"
+		(property "Footprint" "Connector_PinHeader_2.54mm:PinHeader_1x03_P2.54mm_Vertical"
 			(at 450.85 241.3 0)
 			(effects
@@
 			)
 		)
-		(property "Footprint" "Library:PinHeader_1x04_P2.54mm_Vertical"
+		(property "Footprint" "Connector_PinHeader_2.54mm:PinHeader_1x04_P2.54mm_Vertical"
 			(at 447.04 340.36 0)
 			(effects

Commit message: .
Parts:
- removed J3: Conn_01x04_Socket, Connector_PinHeader_2.54mm:PinHeader_1x04_P2.54mm_Vertical, symbol Library:Conn_01x04_Socket
- removed J5: Conn_01x02_Socket, Library:SolderWirePad_1x02_SMD_3x4mm, symbol Library:Conn_01x02_Socket
- added J3: Conn_01x04_Pin, Connector_PinHeader_2.54mm:PinHeader_1x04_P2.54mm_Vertical, symbol Library:Conn_01x04_Pin
- added J5: Conn_01x02_Pin, Connector_PinHeader_2.54mm:PinHeader_1x02_P2.54mm_Vertical, symbol Library:Conn_01x02_Pin
Connections:
- net GND_MCU: now also J3.2 (Pin_2)
- net IR_RX: now also J3.3 (Pin_3)
- net IR_TX: now also J5.2 (Pin_2)
- net VUSB: now also J3.4 (Pin_4)
- new net GLo: J3.1 (Pin_1), J5.1 (Pin_1)

Commit message: .
Connections:
- net PWM_ANG_I: now also U14.2 (IN1); no longer U14.3 (IN2)
- net PWM_ANG_O: now also U14.7 (OUT1); no longer U14.6 (OUT2)
- net PWM_GRB_I: now also U14.3 (IN2); no longer U14.2 (IN1)
- net PWM_GRB_O: now also U14.6 (OUT2); no longer U14.7 (OUT1)
- net VUSB: now also U5.3 (EN)
Changed lines of the file:
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@@
 	)
 	(junction
+		(at 195.58 219.71)
+		(diameter 0)
+		(color 0 0 0 0)
+	)
+	(junction
 		(at 294.64 288.29)
 		(diameter 0)
@@
 	(wire
 		(pts
+			(xy 195.58 219.71) (xy 196.85 219.71)
+		)
+		(stroke
+			(width 0)
+			(type default)
+		)
+	)
+	(wire
+		(pts
 			(xy 488.95 129.54) (xy 499.11 129.54)
 		)
@@
 	(wire
 		(pts
+			(xy 195.58 219.71) (xy 195.58 224.79)
+		)
+		(stroke
+			(width 0)
+			(type default)
+		)
+	)
+	(wire
+		(pts
 			(xy 349.25 358.14) (xy 351.79 358.14)
 		)
@@
 	(wire
 		(pts
+			(xy 196.85 224.79) (xy 195.58 224.79)
+		)
+		(stroke
+			(width 0)
+			(type default)
+		)
+	)
+	(wire
+		(pts
 			(xy 223.52 217.17) (xy 223.52 219.71)
 		)
@@
 	(wire
 		(pts
-			(xy 190.5 219.71) (xy 196.85 219.71)
+			(xy 190.5 219.71) (xy 195.58 219.71)
 		)
 		(stroke
@@
 		)
 	)
-	(label "PWM_ANG_I"
-		(at 527.05 153.67 180)
-		(effects
-			(font
-				(size 1.27 1.27)
-			)
-			(justify right bottom)
-		)
-	)
 	(label "5V_MOT"
 		(at 510.54 184.15 0)
@@
 		)
 	)
+	(label "PWM_ANG_I"
+		(at 527.05 151.13 180)
+		(effects
+			(font
+				(size 1.27 1.27)
+			)
+			(justify right bottom)
+		)
+	)
 	(label "D-"
 		(at 355.6 186.69 0)
@@
 		)
 	)
+	(label "PWM_GRB_I"
+		(at 527.05 153.67 180)
+		(effects
+			(font
+				(size 1.27 1.27)
+			)
+			(justify right bottom)
+		)
+	)
 	(label "E_M1_A"
 		(at 436.88 280.67 180)
@@
 		)
 	)
-	(label "PWM_GRB_I"
-		(at 527.05 151.13 180)
-		(effects
-			(font
-				(size 1.27 1.27)
-			)
-			(justify right bottom)
-		)
-	)
 	(label "VUSB"
 		(at 49.53 128.27 0)
@@
 	)
 	(label "PWM_GRB_O"
-		(at 553.72 151.13 0)
+		(at 553.72 153.67 0)
 		(effects
 			(font
@@
 		)
 	)
-	(label "PWM_ANG_O"
-		(at 553.72 153.67 0)
-		(effects
-			(font
-				(size 1.27 1.27)
-			)
-			(justify left bottom)
-		)
-	)
 	(label "5V_MOT"
 		(at 501.65 129.54 0)
@@
 		)
 	)
+	(label "PWM_ANG_O"
+		(at 553.72 151.13 0)
+		(effects
+			(font
+				(size 1.27 1.27)
+			)
+			(justify left bottom)
+		)
+	)

Commit message: .
Parts:
- J2: footprint Library:SolderWirePad_1x02_SMD_3x4mm -> Library:SolderWirePad_1x02_SMD_3x4mm_power
Changed lines of the file:
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@@
 			)
 		)
-		(property "Footprint" "Library:SolderWirePad_1x02_SMD_3x4mm"
+		(property "Footprint" "Library:SolderWirePad_1x02_SMD_3x4mm_power"
 			(at 35.56 193.04 0)
 			(effects

Commit message: .
Parts:
- R6: value 68R -> 20R
Connections:
- net +3.3V: now also J3.4 (Pin_4), R6.1
- net VUSB: no longer J3.4 (Pin_4), R6.1
Other:
- note added: "Changed from VUSB input to 3.3V. Resistor value changed from 68 to 20 ohm"
- note added: "Supply changed from VUSB to 3.3V for IS471FE"
Changed lines of the file:
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@@
 		)
 	)
+	(text "Supply changed from VUSB to 3.3V for IS471FE\n"
+		(exclude_from_sim no)
+		(at 449.326 359.664 0)
+		(effects
+			(font
+				(size 1.27 1.27)
+			)
+		)
+	)
 	(text "gpio_input"
 		(exclude_from_sim no)
@@
 	(text "FROM IR RX (IS471FE)"
 		(exclude_from_sim no)
-		(at 440.182 332.994 0)
+		(at 444.246 332.994 0)
+		(effects
+			(font
+				(size 1.27 1.27)
+			)
+		)
+	)
+	(text "Changed from VUSB input to 3.3V.\n Resistor value changed from 68 to 20 ohm"
+		(exclude_from_sim no)
+		(at 135.636 125.476 0)
 		(effects
 			(font
@@
 	(wire
 		(pts
-			(xy 129.54 143.51) (xy 124.46 143.51)
+			(xy 425.45 337.82) (xy 441.96 337.82)
+		)
+		(stroke
+			(width 0)
+			(type default)
+		)
+	)
+	(wire
+		(pts
+			(xy 129.54 143.51) (xy 120.65 143.51)
 		)
 		(stroke
@@
 	(wire
 		(pts
-			(xy 435.61 337.82) (xy 441.96 337.82)
-		)
-		(stroke
-			(width 0)
-			(type default)
-		)
-	)
-	(wire
-		(pts
 			(xy 321.31 147.32) (xy 321.31 158.75)
 		)
@@
 		)
 	)
-	(label "VUSB"
-		(at 435.61 337.82 180)
-		(effects
-			(font
-				(size 1.27 1.27)
-			)
-			(justify right bottom)
-		)
-	)
 	(label "D+"
 		(at 80.01 143.51 0)
@@
 		)
 	)
-	(label "VUSB"
-		(at 124.46 143.51 180)
-		(effects
-			(font
-				(size 1.27 1.27)
-			)
-			(justify right bottom)
-		)
-	)
 	(label "M1_DIR_I"
 		(at 444.5 189.23 180)
@@
 			)
 		)
-		(property "Value" "68R"
+		(property "Value" "20R"
 			(at 133.35 139.7 90)
 			(effects
@@
 	)
 	(symbol
+		(lib_id "Library:+3.3V")
+		(at 425.45 337.82 0)
+		(unit 1)
+		(exclude_from_sim no)
+		(in_bom yes)
+		(on_board yes)
+		(dnp no)
+		(fields_autoplaced yes)
+		(property "Reference" "#PWR046"
+			(at 425.45 341.63 0)
+			(effects
+				(font
+					(size 1.27 1.27)
+				)
+				(hide yes)
+			)
+		)
+		(property "Value" "+3.3V"
+			(at 425.45 332.74 0)
+			(effects
+				(font
+					(size 1.27 1.27)
+				)
+			)
+		)
+		(property "Footprint" ""
+			(at 425.45 337.82 0)
+			(effects
+				(font
+					(size 1.27 1.27)
+				)
+				(hide yes)
+			)
+		)
+		(property "Datasheet" ""
+			(at 425.45 337.82 0)
+			(effects
+				(font
+					(size 1.27 1.27)
+				)
+				(hide yes)
+			)
+		)
+		(property "Description" "Power symbol creates a global label with name \"+3.3V\""
+			(at 425.45 337.82 0)
+			(effects
+				(font
+					(size 1.27 1.27)
+				)
+				(hide yes)
+			)
+		)
+		(pin "1"
+		)
+		(instances
+			(project "picr_1_9tdi"
+				(path "/f4c3b324-9d8f-4d10-8101-dec9d8880fba"
+					(reference "#PWR046")
+					(unit 1)
+				)
+			)
+		)
+	)
+	(symbol
 		(lib_id "Library:C")
 		(at 426.72 195.58 0)
@@
 					(unit 1)
 				)
+			)
+		)
+	)
+	(symbol
+		(lib_id "Library:+3.3V")
+		(at 120.65 143.51 0)
+		(unit 1)
+		(exclude_from_sim no)
+		(in_bom yes)
+		(on_board yes)
+		(dnp no)
+		(fields_autoplaced yes)
+		(property "Reference" "#PWR045"
+			(at 120.65 147.32 0)
+			(effects
+				(font
+					(size 1.27 1.27)
+				)
+				(hide yes)
+			)
+		)
+		(property "Value" "+3.3V"
+			(at 120.65 138.43 0)
+			(effects
+				(font
+					(size 1.27 1.27)
+				)
+			)
+		)
+		(property "Footprint" ""
+			(at 120.65 143.51 0)
+			(effects
+				(font
+					(size 1.27 1.27)
+				)
+				(hide yes)
+			)
+		)
+		(property "Datasheet" ""
+			(at 120.65 143.51 0)
+			(effects
+				(font
+					(size 1.27 1.27)
+				)
+				(hide yes)
+			)
+		)
+		(property "Description" "Power symbol creates a global label with name \"+3.3V\""
+			(at 120.65 143.51 0)
+			(effects
+				(font
+					(size 1.27 1.27)
+				)
+				(hide yes)
+			)
+		)
+		(pin "1"
+		)
+		(instances
+			(project "picr_1_9tdi"
+				(path "/f4c3b324-9d8f-4d10-8101-dec9d8880fba"
+					(reference "#PWR045")
+					(unit 1)
+				)

Commit message: .
Parts:
- U3: footprint Library:SOT-583-8 -> Package_TO_SOT_SMD:SOT-583-8
Changed lines of the file:
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@@
 			)
 		)
-		(property "Footprint" "Library:SOT-583-8"
+		(property "Footprint" "Package_TO_SOT_SMD:SOT-583-8"
 			(at 113.03 213.36 0)
 			(effects
