File: electronics/picr_1_9tdi.kicad_pcb (KiCad board)
At the start: 4 copper layers, 50 x 50 mm, 75 parts, among them J1 Conn_01x03_Pin, J2 10118193-0001LF, J3 Conn_01x02_Socket, J4 Conn_01x02_Socket, J5 Conn_01x02_Socket, J6 Conn_01x02_Socket, J7 Conn_01x02_Socket, J9 Conn_01x02_Socket, Q1 BSC026N08NS5, U1 PDRV8243SDGQQ1, U10 NCP718BSN500T1G, U11 PDRV8243SDGQQ1, U12 PDRV8243SDGQQ1, U13 215079-4, U2 STM32G441KBT6, U3 CM1223-02SO, U4 MIC5504-3.3YM5, U5 NCP718BSN500T1G, U6 215079-4, U7 215079-4, U8 215079-4, U9 20021121-00010T4LF

Commit message: Schem rev2
Parts:
- moved U9 15.2 mm to (248.0, 73.5)
- moved J7 10.4 mm to (225.0, 35.5)
- moved Q1 7.47 mm to (239.6, 46.4)
Changed lines of the file:
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@@
 	(footprint "Library:SolderWirePad_1x02_SMD_3x4mm"
 		(layer "F.Cu")
-		(at 221.14 45.13)
+		(at 225 35.5)
 		(descr "Wire Pad, Square, SMD Pad,  3mm x 6mm")
 		(tags "MeasurementPoint Square SMDPad 3mmx6mm ")
@@
 		(fp_text user "*"
 			(at -2.3749 -4.622419 0)
-			(unlocked yes)
 			(layer "F.SilkS")
 			(effects
@@
 		(fp_text user "*"
 			(at -1.1684 -3.5179 0)
+			(unlocked yes)
 			(layer "F.Fab")
 			(effects
@@
 		(fp_text user "*"
 			(at -2.3749 -4.622419 0)
-			(unlocked yes)
 			(layer "F.SilkS")
 			(effects
@@
 			)
 		)
-		(fp_text user "${REFERENCE}"
-			(at 0 0 0)
+		(fp_text user "*"
+			(at -1.1684 -3.5179 0)
 			(unlocked yes)
 			(layer "F.Fab")
@@
 			)
 		)
-		(fp_text user "*"
-			(at -1.1684 -3.5179 0)
+		(fp_text user "${REFERENCE}"
+			(at 0 0 0)
+			(unlocked yes)
 			(layer "F.Fab")
 			(effects
@@
 	(footprint "Library:HDR-SMD_10P-P1.27-V-M-R2-C5-S1.27-LS5.5"
 		(layer "F.Cu")
-		(at 232.781 72.525)
+		(at 247.96 73.45)
 		(property "Reference" "U9"
 			(at -0.0635 -3.85 0)
@@
 	(footprint "Library:TDSON-8-1"
 		(layer "F.Cu")
-		(at 232.13 46.19)
+		(at 239.595 46.365)
 		(descr "Power MOSFET package, TDSON-8-1, 5.15x5.9mm (https://www.infineon.com/cms/en/product/packages/PG-TDSON/PG-TDSON-8-1/)")
 		(tags "tdson ")
@@
 		(fp_text user "*"
 			(at -2.3749 -4.622419 0)
-			(unlocked yes)
 			(layer "F.SilkS")
 			(effects
@@
 		(fp_text user "*"
 			(at -1.1684 -3.5179 0)
+			(unlocked yes)
 			(layer "F.Fab")
 			(effects

Commit message: Schem rev3
Parts:
- removed D3: RF-WUB190DS-DD, Library:LED_0201_0603Metric_Pad0.64x0.40mm_HandSolder
- removed the J1 at (234.0, 83.4)
- removed the J1 at (144.0, 116.6)
- removed the Q1 at (149.7, 119.0)
- removed the Q1 at (239.6, 46.4)
- removed U17: ~, Library:SI8640AB-B-IS1
- added C30: 10u, Library:C_0805_2012Metric_Pad1.18x1.45mm_HandSolder, F.Cu at (155.0, 111.3)
- added C31: 0.1u, Library:C_0603_1608Metric_Pad1.08x0.95mm_HandSolder, F.Cu at (127.7, 91.6)
- added C32: 0.1u, Library:C_0603_1608Metric_Pad1.08x0.95mm_HandSolder, F.Cu at (127.7, 94.1)
- added C33: 0.1u, Library:C_0603_1608Metric_Pad1.08x0.95mm_HandSolder, F.Cu at (127.7, 96.7)
- added C34: 0.1u, Library:C_0603_1608Metric_Pad1.08x0.95mm_HandSolder, F.Cu at (127.7, 99.2)
- added C35: 0.1u, Library:C_0603_1608Metric_Pad1.08x0.95mm_HandSolder, F.Cu at (132.1, 76.6)
- added C36: 0.1u, Library:C_0603_1608Metric_Pad1.08x0.95mm_HandSolder, F.Cu at (132.1, 79.1)
- added C37: 0.1u, Library:C_0603_1608Metric_Pad1.08x0.95mm_HandSolder, F.Cu at (132.1, 81.6)
- added C38: 0.1u, Library:C_0603_1608Metric_Pad1.08x0.95mm_HandSolder, F.Cu at (132.1, 84.1)
- added D1: RF-WUB190DS-DD, Library:LED_0201_0603Metric_Pad0.64x0.40mm_HandSolder, F.Cu at (127.7, 116.5)
- added J1: USB_B_Micro_copy, Library:USB_Micro-B_Amphenol_10118193-0001LF_Horizontal, F.Cu at (137.6, 104.8)
- added J8: Conn_01x02_Socket, Library:SolderWirePad_1x02_SMD_3x4mm, F.Cu at (112.9, 100.1)
- added L1: 1.5u, Library:SRP4021HMCT-1R5M_custom, F.Cu at (158.2, 70.2)
- added Q1: AON6411_copy, Library:BUK6Y10-30PX, F.Cu at (160.8, 114.7)
- added R20: 10K, Library:R_0603_1608Metric_Pad0.98x0.95mm_HandSolder, F.Cu at (140.8, 84.1)
- added R21: 10K, Library:R_0603_1608Metric_Pad0.98x0.95mm_HandSolder, F.Cu at (140.8, 86.6)
- added U14: ~, Library:SI8640AB-B-IS1, F.Cu at (148.9, 96.6)
- added U15: MAX12930EASA+, Library:SOIC-8_L4.9-W3.9-P1.27-LS6.0-BL, F.Cu at (158.0, 88.5)
- C1, C12, C14, C16, C17, C22, C27: footprint Library:C_1206_3216Metric_Pad1.33x1.80mm_HandSolder -> Library:C_0805_2012Metric_Pad1.18x1.45mm_HandSolder
- C10, C19, C9: footprint Library:C_1206_3216Metric_Pad1.33x1.80mm_HandSolder -> Library:C_0603_1608Metric_Pad1.08x0.95mm_HandSolder
- C11, C2, C3: value 1u -> 10u; footprint Library:C_1206_3216Metric_Pad1.33x1.80mm_HandSolder -> Library:C_0805_2012Metric_Pad1.18x1.45mm_HandSolder
- C13, C18, C23, C25, C26: value 10u -> 100n; footprint Library:C_1206_3216Metric_Pad1.33x1.80mm_HandSolder -> Library:C_0603_1608Metric_Pad1.08x0.95mm_HandSolder
- C15, C28: value 0.1u -> 100n; footprint Library:C_1206_3216Metric_Pad1.33x1.80mm_HandSolder -> Library:C_0603_1608Metric_Pad1.08x0.95mm_HandSolder
- C20: value 0.1u -> 10u; footprint Library:C_1206_3216Metric_Pad1.33x1.80mm_HandSolder -> Library:C_0603_1608Metric_Pad1.08x0.95mm_HandSolder
- C21: value 10u -> 0.1u; footprint Library:C_1206_3216Metric_Pad1.33x1.80mm_HandSolder -> Library:C_0603_1608Metric_Pad1.08x0.95mm_HandSolder
- C24, C29: value 0.1u -> 10u; footprint Library:C_1206_3216Metric_Pad1.33x1.80mm_HandSolder -> Library:C_0805_2012Metric_Pad1.18x1.45mm_HandSolder
- C4: value 100n -> 10u; footprint Library:C_1206_3216Metric_Pad1.33x1.80mm_HandSolder -> Library:C_0805_2012Metric_Pad1.18x1.45mm_HandSolder
- C5, C7: value 100n -> 1u; footprint Library:C_1206_3216Metric_Pad1.33x1.80mm_HandSolder -> Library:C_0603_1608Metric_Pad1.08x0.95mm_HandSolder
- C6: value 100n -> 0.1u; footprint Library:C_1206_3216Metric_Pad1.33x1.80mm_HandSolder -> Library:C_0603_1608Metric_Pad1.08x0.95mm_HandSolder
- C8: value 1u -> 0.1u; footprint Library:C_1206_3216Metric_Pad1.33x1.80mm_HandSolder -> Library:C_0603_1608Metric_Pad1.08x0.95mm_HandSolder
- J2: value 10118193-0001LF -> Conn_01x02_Socket; footprint Library:USB_Micro-B_Amphenol_10118193-0001LF_Horizontal -> Library:SolderWirePad_1x02_SMD_3x4mm
- J4, J6: value Conn_01x02_Socket -> Conn_01x03_Pin; footprint Library:SolderWirePad_1x02_SMD_3x4mm -> Library:PinHeader_1x03_P2.54mm_Vertical
- R1, R7: value 10K -> 100K; footprint Library:R_0201_0603Metric_Pad0.64x0.40mm_HandSolder -> Library:R_0603_1608Metric_Pad0.98x0.95mm_HandSolder
- R10, R16: value 2K -> 10K; footprint Library:R_0201_0603Metric_Pad0.64x0.40mm_HandSolder -> Library:R_0603_1608Metric_Pad0.98x0.95mm_HandSolder
- R11: value 22K -> 100R; footprint Library:R_0201_0603Metric_Pad0.64x0.40mm_HandSolder -> Library:R_0603_1608Metric_Pad0.98x0.95mm_HandSolder
- R12: value 10K -> 52K3; footprint Library:R_0201_0603Metric_Pad0.64x0.40mm_HandSolder -> Library:R_0603_1608Metric_Pad0.98x0.95mm_HandSolder
- R13, R17, R18, R5, R6: footprint Library:R_0201_0603Metric_Pad0.64x0.40mm_HandSolder -> Library:R_0603_1608Metric_Pad0.98x0.95mm_HandSolder
- R14: value 22K -> 2K7; footprint Library:R_0201_0603Metric_Pad0.64x0.40mm_HandSolder -> Library:R_0603_1608Metric_Pad0.98x0.95mm_HandSolder
- R15: value 500R -> 100K; footprint Library:R_0201_0603Metric_Pad0.64x0.40mm_HandSolder -> Library:R_0603_1608Metric_Pad0.98x0.95mm_HandSolder
- R19: value 500R -> 2K7; footprint Library:R_0201_0603Metric_Pad0.64x0.40mm_HandSolder -> Library:R_0603_1608Metric_Pad0.98x0.95mm_HandSolder
- R2: value 2K -> 22K; footprint Library:R_0201_0603Metric_Pad0.64x0.40mm_HandSolder -> Library:R_0603_1608Metric_Pad0.98x0.95mm_HandSolder
- R3: value 100R -> 10K; footprint Library:R_0201_0603Metric_Pad0.64x0.40mm_HandSolder -> Library:R_0603_1608Metric_Pad0.98x0.95mm_HandSolder
- R4: value 100K -> 2K7; footprint Library:R_0201_0603Metric_Pad0.64x0.40mm_HandSolder -> Library:R_0603_1608Metric_Pad0.98x0.95mm_HandSolder
- R8: value 10K -> 35K; footprint Library:R_0201_0603Metric_Pad0.64x0.40mm_HandSolder -> Library:R_0603_1608Metric_Pad0.98x0.95mm_HandSolder
- R9: value 500R -> 22K; footprint Library:R_0201_0603Metric_Pad0.64x0.40mm_HandSolder -> Library:R_0603_1608Metric_Pad0.98x0.95mm_HandSolder
- U10: value NCP718BSN500T1G -> 215079-4; footprint Library:SOT-23-5 -> Library:TE_Micro-MaTch_215079-4_2x02_P1.27mm_Vertical
- U11, U12: value PDRV8243SDGQQ1 -> 215079-4; footprint Library:VSSOP_SDGQQ1_TEX-L -> Library:TE_Micro-MaTch_215079-4_2x02_P1.27mm_Vertical
- U13: value 215079-4 -> ~; footprint Library:TE_Micro-MaTch_215079-4_2x02_P1.27mm_Vertical -> Library:SI8640AB-B-IS1
- U16: footprint Library:SI8640AB-B-IS1 -> Library:TE_Micro-MaTch_215079-4_2x02_P1.27mm_Vertical
- U2: value STM32G441KBT6 -> CM1223-02SO; footprint Library:LQFP-32_7x7mm_P0.8mm -> Library:SOT-23-5_L2.9-W1.6-P0.95-LS2.8-BR
- U3: value CM1223-02SO -> NCP718BSN500T1G; footprint Library:SOT-23-5_L2.9-W1.6-P0.95-LS2.8-BR -> Library:SOT-23-5
- U5: value NCP718BSN500T1G -> TPS62933; footprint Library:SOT-23-5 -> Library:SOT-583-8
- U6, U7: value 215079-4 -> PDRV8243SDGQQ1; footprint Library:TE_Micro-MaTch_215079-4_2x02_P1.27mm_Vertical -> Library:VSSOP_SDGQQ1_TEX-L
- U8: value 215079-4 -> STM32G441KBT6; footprint Library:TE_Micro-MaTch_215079-4_2x02_P1.27mm_Vertical -> Library:LQFP-32_7x7mm_P0.8mm
- moved J9 129.0 mm to (112.9, 107.7)
- moved J7 125.8 mm to (112.9, 92.6)
- moved U5 119.8 mm to (127.9, 113.8)
- moved U10 110.0 mm to (124.6, 68.8)
- moved U2 106.2 mm to (123.3, 113.8)
- moved U8 99.4 mm to (126.9, 106.1)
- moved C18 96.4 mm to (123.4, 96.7)
- moved C19 96.1 mm to (123.4, 99.2)
- moved R16 95.0 mm to (136.4, 99.2)
- moved R15 94.8 mm to (136.4, 96.7)
- moved C25 94.6 mm to (127.7, 84.1)
- moved C26 94.3 mm to (127.7, 86.6)
- moved C28 93.1 mm to (127.7, 89.1)
- moved U9 92.3 mm to (158.6, 96.7)
- moved R6 92.0 mm to (132.1, 99.2)
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Connections:
- C1 pad 1: +3.3V -> /VBAT
- C1 pad 2: GND1 -> GND_MOT
- C10 pad 1: /VBAT -> +3.3V
- C10 pad 2: GND1 -> GND_MCU
- C11 pad 1: +5V -> /VBAT
- C11 pad 2: GND1 -> GND_MOT
- C12 pad 2: GND2 -> GND_MOT
- C13 pad 2: GND2 -> GND_MOT
- C14 pad 2: GND2 -> GND_MOT
- C15 pad 1: /VBAT -> Net-(U5-SS)
- C15 pad 2: GND2 -> GND_MOT
- C16 pad 2: GND2 -> GND_MOT
- C17 pad 2: GND2 -> GND_MOT
- C18 pad 1: /VBAT -> Net-(U5-BST)
- C18 pad 2: GND2 -> Net-(U5-SW)
- C19 pad 2: GND2 -> GND_MOT
- C2 pad 1: +5V -> /VBAT
- C2 pad 2: GND1 -> GND_MOT
- C20 pad 1: /VBAT -> /V_SERVO
- C20 pad 2: GND2 -> GND_MOT
- C21 pad 2: GND2 -> GND_MOT
- C22 pad 1: /VBAT -> +3.3V
- C22 pad 2: GND2 -> GND_MCU
- C23 pad 1: /VBAT -> +3.3V
- C23 pad 2: GND2 -> GND_MCU
- C24 pad 2: GND2 -> GND_MOT
- C25 pad 1: /VBAT -> +3.3V
- C25 pad 2: GND2 -> GND_MCU
- C26 pad 1: /VBAT -> /NRST
- C26 pad 2: GND2 -> GND_MCU
- C27 pad 2: GND2 -> GND_MOT
- C28 pad 1: /VBAT -> +3.3V
- C28 pad 2: GND2 -> GND_MCU
- C29 pad 2: GND2 -> GND_MOT
- C3 pad 1: +3.3V -> /VBAT
- C3 pad 2: GND1 -> GND_MOT
- C4 pad 1: +3.3V -> /VBAT
- C4 pad 2: GND1 -> GND_MOT
- C5 pad 1: +3.3V -> /VBAT
- C5 pad 2: GND1 -> GND_MOT
- C6 pad 1: +3.3V -> /VBAT
- C6 pad 2: GND1 -> GND_MOT
- C7 pad 1: /NRST -> /VUSB
- C7 pad 2: GND1 -> GND_MCU
- C8 pad 2: GND1 -> GND_MOT
- C9 pad 1: /V_SERVO -> /5V_MOT
- C9 pad 2: GND1 -> GND_MOT
- J2 pad 1: +5V -> /VBAT_IN
- J2 pad 2: unconnected-(J2-ID-Pad2) -> GND_MOT
- J3 pad 1: /M1_OUT1 -> /IR_RX
- J3 pad 2: /M1_OUT2 -> GND_MCU
- J4 pad 1: /M2_OUT1 -> /PWM_GRB_O
- J4 pad 2: /M2_OUT2 -> /V_SERVO
- J5 pad 1: /M3_OUT1 -> /IR_TX
- J5 pad 2: /M3_OUT2 -> GND_MCU
- J6 pad 1: /VBAT_IN -> /PWM_ANG_O
- J6 pad 2: GND1 -> /V_SERVO
- J7 pad 1: /IR_TX -> /M3_OUT1
- J7 pad 2: GND1 -> /M3_OUT2
- J9 pad 1: /IR_RX -> /M2_OUT1
- J9 pad 2: GND1 -> /M2_OUT2
- R1 pad 1: GND1 -> GND_MOT
- R1 pad 2: Net-(U2-BOOT0) -> Net-(U1-ITRIP)
- R10 pad 1: GND2 -> Net-(U6-DRVOFF)
- R10 pad 2: Net-(U11-ITRIP) -> GND_MOT
- R11 pad 1: Net-(U11-SR) -> /VUSB
- R11 pad 2: GND2 -> Net-(D1-A)
- R12 pad 1: Net-(U1-DRVOFF) -> /V_SERVO
- R12 pad 2: GND2 -> Net-(U5-FB)
- R13 pad 1: Net-(U11-DRVOFF) -> Net-(U5-FB)
- R13 pad 2: GND2 -> GND_MOT
- R14 pad 1: Net-(U1-SR) -> Net-(U6-IPROPI)
- R14 pad 2: GND2 -> GND_MOT
- R15 pad 1: Net-(U11-IPROPI) -> GND_MOT
- R15 pad 2: GND2 -> Net-(U7-ITRIP)
- R16 pad 1: GND2 -> GND_MCU
- R16 pad 2: Net-(U12-ITRIP) -> Net-(U8-PB8)
- R17 pad 1: Net-(U12-SR) -> Net-(U7-SR)
- R17 pad 2: GND2 -> GND_MOT
- R18 pad 1: Net-(U12-DRVOFF) -> Net-(U7-DRVOFF)
- R18 pad 2: GND2 -> GND_MOT
- R19 pad 1: Net-(U12-IPROPI) -> Net-(U7-IPROPI)
- R19 pad 2: GND2 -> GND_MOT
- R2 pad 1: GND2 -> Net-(U1-SR)
- R2 pad 2: Net-(U1-ITRIP) -> GND_MOT
- R3 pad 1: +5V -> Net-(U1-DRVOFF)
- R3 pad 2: /IR_TX -> GND_MOT
- R4 pad 1: +5V -> Net-(U1-IPROPI)
- R4 pad 2: /IR_RX -> GND_MOT
- R5 pad 1: +5V -> /VUSB
- R5 pad 2: Net-(D3-A) -> /IR_TX
- R6 pad 1: /VBAT_IN -> /VUSB
- R6 pad 2: GND1 -> /IR_RX
- R7 pad 1: +5V -> GND_MOT
- R7 pad 2: Net-(U17-EN2) -> Net-(U6-ITRIP)
- R8 pad 1: +5V -> Net-(U5-RT)
- R8 pad 2: Net-(U16-EN2) -> GND_MOT
- R9 pad 1: Net-(U1-IPROPI) -> Net-(U6-SR)
- R9 pad 2: GND2 -> GND_MOT
- U1 pad 12: GND2 -> GND_MOT
- U1 pad 13: GND2 -> GND_MOT
- U1 pad 14: GND2 -> GND_MOT
- U1 pad 15: GND2 -> GND_MOT
- U1 pad 16: GND2 -> GND_MOT
- U1 pad 17: GND2 -> GND_MOT
- U1 pad 2: GND2 -> GND_MOT
- U1 pad 26: GND2 -> GND_MOT
- U1 pad 27: GND2 -> GND_MOT
- U1 pad EPAD: GND2 -> GND_MOT
- U10 pad 1: /VBAT -> GND_MCU
- U10 pad 2: GND1 -> +3.3V
- U10 pad 3: /VBAT -> /E_M1_A
- U10 pad 4: unconnected-(U10-NC-Pad4) -> /E_M1_B
- U11 pad 1: Net-(U11-SR) -> GND_MCU
- U11 pad 2: GND2 -> +3.3V
- U11 pad 3: /M2_DIR_O -> /E_M2_A
- U11 pad 4: /PWM_M2_O -> /E_M2_B
- U12 pad 1: Net-(U12-SR) -> GND_MCU
- U12 pad 2: GND2 -> +3.3V
- U12 pad 3: /M3_DIR_O -> /E_M3_A
- U12 pad 4: /PWM_M3_O -> /E_M3_B
- U13 pad 1: GND1 -> +3.3V
- U13 pad 2: +3.3V -> GND_MCU
- U13 pad 3: /E_M1_A -> /PWM_M1_I
- U13 pad 4: /E_M1_B -> /PWM_M2_I
- U16 pad 1: +3.3V -> GND_MOT
- U16 pad 2: GND1 -> /PWM_TH_O
- U16 pad 3: /PWM_M1_I -> unconnected-(U16-Pad3)
- U16 pad 4: /PWM_M2_I -> unconnected-(U16-Pad4)
- U2 pad 1: +3.3V -> unconnected-(U2-NC-Pad1)
- U2 pad 2: unconnected-(U2-PF0-Pad2) -> GND_MCU
- U2 pad 3: unconnected-(U2-PF1-Pad3) -> /D+
- U2 pad 4: /NRST -> /D-
- U2 pad 5: /E_M1_A -> /VUSB
- U3 pad 1: unconnected-(U3-NC-Pad1) -> /VBAT
- U3 pad 2: GND1 -> GND_MOT
- U3 pad 3: /D+ -> /VBAT
- U3 pad 4: /D- -> unconnected-(U3-NC-Pad4)
- U3 pad 5: +5V -> /5V_MOT
- U4 pad 1: +5V -> /VUSB
- U4 pad 2: GND1 -> GND_MCU
- U5 pad 1: /VBAT -> Net-(U5-RT)
- U5 pad 2: GND1 -> unconnected-(U5-EN-Pad2)
- U5 pad 4: unconnected-(U5-NC-Pad4) -> GND_MOT
- U5 pad 5: +5V -> Net-(U5-SW)
- U6 pad 1: GND1 -> Net-(U6-SR)
- U6 pad 2: +3.3V -> GND_MOT
- U6 pad 3: /E_M2_A -> /M2_DIR_O
- U6 pad 4: /E_M2_B -> /PWM_M2_O
- U7 pad 1: GND1 -> Net-(U7-SR)
- U7 pad 2: +3.3V -> GND_MOT
- U7 pad 3: /E_M3_A -> /M3_DIR_O
- U7 pad 4: /E_M3_B -> /PWM_M3_O
- U8 pad 1: /PWM_TH_O -> +3.3V
- U8 pad 3: GND1 -> /IR_RX
- U8 pad 4: unconnected-(U8-ENC_B-Pad4) -> /NRST
- U9 pad 3: GND1 -> GND_MCU
- U9 pad 5: GND1 -> GND_MCU
- U9 pad 9: GND1 -> GND_MCU
Routing:
- net /D-: track 9.26 -> 0.00 mm
- net /D+: track 9.24 -> 0.00 mm
Other:
- board outline removed

Commit message: .
Parts:
- removed the C28 at (127.7, 89.1)
- added C12: 10u, Library:C_0603_1608Metric_Pad1.08x0.95mm_HandSolder, F.Cu at (49.6, 41.5)
- added C27: 100n, Library:C_0603_1608Metric_Pad1.08x0.95mm_HandSolder, F.Cu at (174.3, 99.8)
- added C34: 0.1u, Library:C_0603_1608Metric_Pad1.08x0.95mm_HandSolder, F.Cu at (49.6, 44.0)
- added C35: 0.1u, Library:C_0603_1608Metric_Pad1.08x0.95mm_HandSolder, F.Cu at (49.6, 46.5)
- added J3: Conn_01x03_Pin, Library:PinHeader_1x03_P2.54mm_Vertical, F.Cu at (203.8, 84.1)
- D1: footprint Library:LED_0201_0603Metric_Pad0.64x0.40mm_HandSolder -> Library:LED_0603_1608Metric_Pad1.05x0.95mm_HandSolder
- R12: renamed from R11; value 100R -> 4K7
- R4: renamed from R8; value 35K -> 10K
- R6: renamed from R5; value 100R -> 68R
- U10: renamed from U11; moved to B.Cu
- U11: renamed from U12; moved to B.Cu
- U15: renamed from U16; moved to B.Cu
- U9: renamed from U10; moved to B.Cu
- moved Q1 106.8 mm to (55.5, 96.9)
- moved C21 96.4 mm to (59.3, 82.1)
- moved U8 86.9 mm to (72.7, 83.4), turned to 180 degrees
- moved U5 84.6 mm to (81.3, 76.8)
- moved J1 75.8 mm to (69.2, 72.3), turned to -90 degrees
- moved U15 75.7 mm to (75.5, 52.6), turned to -90 degrees
- moved U1 74.8 mm to (79.2, 112.0)
- moved C1 73.5 mm to (75.1, 123.8), turned to -90 degrees
- moved C2 70.7 mm to (77.1, 123.8), turned to -90 degrees
- moved U12 69.9 mm to (79.2, 93.0), turned to 180 degrees
- moved U4 69.3 mm to (92.7, 112.0)
- moved C4 67.4 mm to (79.1, 123.8), turned to -90 degrees
- moved C3 66.1 mm to (81.1, 123.8), turned to -90 degrees
- moved J2 64.9 mm to (58.5, 105.3), turned to -90 degrees
- moved U6 64.1 mm to (106.1, 112.0)
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- renumbered C18 to C10, C20 to C11, C12 to C13, C16 to C15, C7 to C16, C10 to C18, C21 to C20, C22 to C21, C23 to C22, C24 to C23, C25 to C24, C26 to C25, C27 to C26, C29 to C28, C30 to C29, C31 to C30, C32 to C31, C34 to C32, C37 to C36, C38 to C37, C11 to C5, C13 to C6, C6 to C7, C15 to C8, C8 to C9, R9 to R10, R10 to R11, R14 to R13, R15 to R14, R16 to R15, R17 to R16, R18 to R17, R19 to R18, R20 to R19, R21 to R20, R4 to R5, R12 to R7, R13 to R8, R7 to R9, U13 to U12, U14 to U13, U15 to U14, U5 to U3, U6 to U4, U4 to U5, U7 to U6, U8 to U7, U9 to U8
Connections:
- C11 pad 1: /V_SERVO -> /5V_MOT
- J4 pad 2: /V_SERVO -> /5V_MOT
- J6 pad 2: /V_SERVO -> /5V_MOT
- L1 pad 2: /V_SERVO -> /5V_MOT
- Q1 pad 1: /VBAT_IN -> /VBAT
- Q1 pad 2: /VBAT_IN -> /VBAT
- Q1 pad 3: /VBAT_IN -> /VBAT
- Q1 pad 5: /VBAT -> /VBAT_IN
- R19 pad 1: Net-(C35-Pad2) -> /5V_MOT
- R20 pad 1: Net-(C36-Pad2) -> /5V_MOT
- R7 pad 1: /V_SERVO -> /5V_MOT
Routing:
- net /PWM_TH_I: track 0.00 -> 19.9 mm, vias 0 -> 2
- net /PWM_M3_I: track 0.00 -> 18.6 mm, vias 0 -> 2
- net /PWM_M2_I: track 0.00 -> 17.6 mm, vias 0 -> 2
- net /M_NSLEEP_I: track 0.00 -> 17.5 mm, vias 0 -> 2
- net /M1_DIR_I: track 0.00 -> 17.5 mm, vias 0 -> 2
- net /M3_DIR_I: track 0.00 -> 17.1 mm, vias 0 -> 2
- net /PWM_M1_I: track 0.00 -> 16.4 mm
- net /M2_DIR_I: track 0.00 -> 16.4 mm
- net /PWM_GRB_I: track 0.00 -> 6.17 mm, vias 0 -> 2
- net /PWM_ANG_I: track 0.00 -> 5.74 mm
- net /VUSB: track 0.00 -> 1.76 mm
- net GND_MOT: track 0.00 -> 0.77 mm
Other:
- board outline added: 50 x 50 mm

Commit message: .
Connections:
- R12 pad 1: /VUSB -> /MCU_LED
- U7 pad 26: unconnected-(U7-PB3-Pad26) -> /MCU_LED
Changed lines of the file:
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@@
 	(net 62 "/SWCLK")
 	(net 63 "/E_M1_A")
-	(net 64 "unconnected-(U7-PB3-Pad26)")
+	(net 64 "/MCU_LED")
 	(net 65 "/E_M2_A")
 	(net 66 "/PWM_ANG_I")
@@
 		(tags "capacitor handsolder")
 		(property "Reference" "C2"
-			(at 2.7625 -0.1 0)
+			(at 0 -1.68 270)
 			(layer "F.SilkS")
 			(effects
@@
 		)
 		(property "Value" "10u"
-			(at 0 1.68 90)
+			(at 0 1.68 270)
 			(layer "F.Fab")
 			(effects
@@
 		)
 		(property "Datasheet" "~"
-			(at 0 0 90)
+			(at 0 0 270)
 			(layer "F.Fab")
 			(hide yes)
@@
 		)
 		(property "Description" "Unpolarized capacitor"
-			(at 0 0 90)
+			(at 0 0 270)
 			(layer "F.Fab")
 			(hide yes)
@@
 		)
 		(fp_text user "${REFERENCE}"
-			(at 0 0 90)
+			(at 0 0 270)
 			(layer "F.Fab")
 			(effects
@@
 		(tags "capacitor handsolder")
 		(property "Reference" "C22"
-			(at 0.2875 1.45 0)
+			(at 0 -1.43 180)
 			(layer "F.SilkS")
 			(effects
@@
 		)
 		(property "Value" "100n"
-			(at 0 1.43 0)
+			(at 0 1.43 180)
 			(layer "F.Fab")
 			(effects
@@
 		)
 		(property "Datasheet" "~"
-			(at 0 0 0)
+			(at 0 0 180)
 			(layer "F.Fab")
 			(hide yes)
@@
 		)
 		(property "Description" "Unpolarized capacitor"
-			(at 0 0 0)
+			(at 0 0 180)
 			(layer "F.Fab")
 			(hide yes)
@@
 		)
 		(fp_text user "${REFERENCE}"
-			(at 0 0 0)
+			(at 0 0 180)
 			(layer "F.Fab")
 			(effects
@@
 		(tags "capacitor handsolder")
 		(property "Reference" "C16"
-			(at 0 1.45 90)
+			(at 0 -1.43 270)
 			(layer "F.SilkS")
 			(effects
@@
 		)
 		(property "Value" "1u"
-			(at 0 1.43 90)
+			(at 0 1.43 270)
 			(layer "F.Fab")
 			(effects
@@
 		)
 		(property "Datasheet" "~"
-			(at 0 0 90)
+			(at 0 0 270)
 			(layer "F.Fab")
 			(hide yes)
@@
 		)
 		(property "Description" "Unpolarized capacitor"
-			(at 0 0 90)
+			(at 0 0 270)
 			(layer "F.Fab")
 			(hide yes)
@@
 		)
 		(fp_text user "${REFERENCE}"
-			(at 0 0 90)
+			(at 0 0 270)
 			(layer "F.Fab")
 			(effects
@@
 		(tags "capacitor handsolder")
 		(property "Reference" "C24"
-			(at 3.3375 -0.1 0)
+			(at 0 -1.43 180)
 			(layer "F.SilkS")
 			(effects
@@
 		)
 		(property "Value" "100n"
-			(at 0 1.43 0)
+			(at 0 1.43 180)
 			(layer "F.Fab")
 			(effects
@@
 		)
 		(property "Datasheet" "~"
-			(at 0 0 0)
+			(at 0 0 180)
 			(layer "F.Fab")
 			(hide yes)
@@
 		)
 		(property "Description" "Unpolarized capacitor"
-			(at 0 0 0)
+			(at 0 0 180)
 			(layer "F.Fab")
 			(hide yes)
@@
 		)
 		(fp_text user "${REFERENCE}"
-			(at 0 0 0)
+			(at 0 0 180)
 			(layer "F.Fab")
 			(effects
@@
 		(tags "capacitor handsolder")
 		(property "Reference" "C4"
-			(at 2.6375 -0.1 0)
+			(at 0 -1.68 270)
 			(layer "F.SilkS")
 			(effects
@@
 		)
 		(property "Value" "10u"
-			(at 0 1.68 90)
+			(at 0 1.68 270)
 			(layer "F.Fab")
 			(effects
@@
 		)
 		(property "Datasheet" "~"
-			(at 0 0 90)
+			(at 0 0 270)
 			(layer "F.Fab")
 			(hide yes)
@@
 		)
 		(property "Description" "Unpolarized capacitor"
-			(at 0 0 90)
+			(at 0 0 270)
 			(layer "F.Fab")
 			(hide yes)
@@
 		)
 		(fp_text user "${REFERENCE}"
-			(at 0 0 90)
+			(at 0 0 270)
 			(layer "F.Fab")
 			(effects
@@
 		(tags "Through hole pin header THT 1x03 2.54mm single row")
 		(property "Reference" "J4"
-			(at 3.3 5.04 0)
+			(at 0 -2.38 180)
 			(layer "F.SilkS")
 			(effects
@@
 		)
 		(property "Value" "Conn_01x03_Pin"
-			(at 0 7.46 0)
+			(at 0 7.46 180)
 			(layer "F.Fab")
 			(effects
@@
 		)
 		(property "Datasheet" "~"
-			(at 0 0 0)
+			(at 0 0 180)
 			(layer "F.Fab")
 			(hide yes)
@@
 		)
 		(property "Description" "Generic connector, single row, 01x03, script generated"
-			(at 0 0 0)
+			(at 0 0 180)
 			(layer "F.Fab")
 			(hide yes)
@@
 		)
 		(fp_text user "${REFERENCE}"
-			(at 0 2.54 90)
+			(at 0 2.54 270)
 			(layer "F.Fab")
 			(effects
@@
 			(layers "F.Cu" "F.Mask" "F.Paste")
 			(roundrect_rratio 0.25)
-			(net 64 "unconnected-(U7-PB3-Pad26)")
+			(net 64 "/MCU_LED")
 			(pinfunction "PB3")
-			(pintype "no_connect")
+			(pintype "passive")
 		)
 		(pad "27" smd roundrect
@@
 		(tags "capacitor handsolder")
 		(property "Reference" "C25"
-			(at 0 -1.43 90)
+			(at 0 -1.43 270)
 			(layer "F.SilkS")
 			(effects
@@
 		)
 		(property "Value" "100n"
-			(at 0 1.43 90)
+			(at 0 1.43 270)
 			(layer "F.Fab")
 			(effects
@@
 		)
 		(property "Datasheet" "~"
-			(at 0 0 90)
+			(at 0 0 270)
 			(layer "F.Fab")
 			(hide yes)
@@
 		)
 		(property "Description" "Unpolarized capacitor"
-			(at 0 0 90)
+			(at 0 0 270)
 			(layer "F.Fab")
 			(hide yes)
@@
 		)
 		(fp_text user "${REFERENCE}"
-			(at 0 0 90)
+			(at 0 0 270)
 			(layer "F.Fab")
 			(effects
@@
 			(layers "F.Cu" "F.Mask" "F.Paste")
 			(roundrect_rratio 0.25)
-			(net 4 "/VUSB")
+			(net 64 "/MCU_LED")
 			(pintype "passive")
 		)
@@
 		(tags "capacitor handsolder")
 		(property "Reference" "C1"
-			(at 2.7625 0 180)
+			(at 0 -1.68 270)
 			(layer "F.SilkS")
 			(effects
@@
 		)
 		(property "Value" "10u"
-			(at 0 1.68 90)
+			(at 0 1.68 270)
 			(layer "F.Fab")
 			(effects
@@
 		)
 		(property "Datasheet" "~"
-			(at 0 0 90)
+			(at 0 0 270)
 			(layer "F.Fab")
 			(hide yes)
@@
 		)
 		(property "Description" "Unpolarized capacitor"
-			(at 0 0 90)
+			(at 0 0 270)
 			(layer "F.Fab")
 			(hide yes)
@@
 		)
 		(fp_text user "${REFERENCE}"
-			(at 0 0 90)
+			(at 0 0 270)
 			(layer "F.Fab")
 			(effects
@@
 		(tags "capacitor handsolder")
 		(property "Reference" "C3"
-			(at 2.6375 -0.1 0)
+			(at 0 -1.68 270)
 			(layer "F.SilkS")
 			(effects
@@
 		)
 		(property "Value" "10u"
-			(at 0 1.68 90)
+			(at 0 1.68 270)
 			(layer "F.Fab")
 			(effects
@@
 		)
 		(property "Datasheet" "~"
-			(at 0 0 90)
+			(at 0 0 270)
 			(layer "F.Fab")
 			(hide yes)
@@
 		)
 		(property "Description" "Unpolarized capacitor"
-			(at 0 0 90)
+			(at 0 0 270)
 			(layer "F.Fab")
 			(hide yes)
@@
 		)
 		(fp_text user "${REFERENCE}"
-			(at 0 0 90)
+			(at 0 0 270)
 			(layer "F.Fab")
 			(effects
@@
 		(tags "Through hole pin header THT 1x03 2.54mm single row")
 		(property "Reference" "J6"
-			(at 3.5 1.34 0)
+			(at 0 -2.38 180)
 			(layer "F.SilkS")
 			(effects
@@
 		)
 		(property "Value" "Conn_01x03_Pin"
-			(at 0 7.46 0)
+			(at 0 7.46 180)
 			(layer "F.Fab")
 			(effects
@@
 		)
 		(property "Datasheet" "~"
-			(at 0 0 0)
+			(at 0 0 180)
 			(layer "F.Fab")
 			(hide yes)
@@
 		)
 		(property "Description" "Generic connector, single row, 01x03, script generated"
-			(at 0 0 0)
+			(at 0 0 180)
 			(layer "F.Fab")
 			(hide yes)
@@
 		)
 		(fp_text user "${REFERENCE}"
-			(at 0 2.54 90)
+			(at 0 2.54 270)
 			(layer "F.Fab")
 			(effects
@@
 		(tags "capacitor handsolder")
 		(property "Reference" "C8"
-			(at 0 -1.43 180)
+			(at 0 -1.43 0)
 			(layer "F.SilkS")
 			(effects
@@
 		)
 		(property "Value" "100n"
-			(at 0 1.43 180)
+			(at 0 1.43 0)
 			(layer "F.Fab")
 			(effects
@@
 		)
 		(property "Datasheet" "~"
-			(at 0 0 180)
+			(at 0 0 0)
 			(layer "F.Fab")
 			(hide yes)
@@
 		)
 		(property "Description" "Unpolarized capacitor"
-			(at 0 0 180)
+			(at 0 0 0)
 			(layer "F.Fab")
 			(hide yes)
@@
 		)
 		(fp_text user "${REFERENCE}"
-			(at 0 0 180)
+			(at 0 0 0)
 			(layer "F.Fab")
 			(effects
@@
 		(tags "capacitor handsolder")
 		(property "Reference" "C18"
-			(at 0 -1.43 90)
+			(at 0 -1.43 270)
 			(layer "F.SilkS")
 			(effects
@@
 		)
 		(property "Value" "1u"
-			(at 0 1.43 90)
+			(at 0 1.43 270)
 			(layer "F.Fab")
 			(effects
@@
 		)
 		(property "Datasheet" "~"
-			(at 0 0 90)
+			(at 0 0 270)
 			(layer "F.Fab")
 			(hide yes)
@@
 		)
 		(property "Description" "Unpolarized capacitor"
-			(at 0 0 90)
+			(at 0 0 270)
 			(layer "F.Fab")
 			(hide yes)
@@
 		)
 		(fp_text user "${REFERENCE}"
-			(at 0 0 90)
+			(at 0 0 270)
 			(layer "F.Fab")
 			(effects

Commit message: .
Parts:
- added J3: Conn_01x04_Socket, Connector_PinHeader_2.54mm:PinHeader_1x04_P2.54mm_Vertical, F.Cu at (212.2, 66.0)
- C1, C13, C14, C15, C17, C2, C21, C23, C26, C28, C29, C3, C4, C5: footprint Library:C_0805_2012Metric_Pad1.18x1.45mm_HandSolder -> Capacitor_SMD:C_0805_2012Metric_Pad1.18x1.45mm_HandSolder
- C10, C22, C24, C25, C27, C6, C8: value 100n -> 0.1u; footprint Library:C_0603_1608Metric_Pad1.08x0.95mm_HandSolder -> Capacitor_SMD:C_0603_1608Metric_Pad1.08x0.95mm_HandSolder
- C11, C12, C16, C18, C19, C20, C30, C31, C32, C33, C34, C35, C36, C37, C7, C9: footprint Library:C_0603_1608Metric_Pad1.08x0.95mm_HandSolder -> Capacitor_SMD:C_0603_1608Metric_Pad1.08x0.95mm_HandSolder
- D1: footprint Library:LED_0603_1608Metric_Pad1.05x0.95mm_HandSolder -> LED_SMD:LED_0603_1608Metric_Pad1.05x0.95mm_HandSolder
- J1: value USB_B_Micro_copy -> 10118193-0001LF
- J2, J7, J8, J9: footprint Library:SolderWirePad_1x02_SMD_3x4mm -> Connector_Wire:SolderWirePad_1x02_SMD_3x4mm
- J4, J6: footprint Library:PinHeader_1x03_P2.54mm_Vertical -> Connector_PinHeader_2.54mm:PinHeader_1x03_P2.54mm_Vertical
- L1: footprint Library:SRP4021HMCT-1R5M_custom -> Inductor_SMD:SRP4021HMCT-1R5M_custom
- Q1: value AON6411_copy -> BUK6Y10-30PX
- R1, R10, R11, R12, R13, R14, R15, R16, R17, R18, R19, R2, R20, R3, R4, R5, R6, R7, R8, R9: footprint Library:R_0603_1608Metric_Pad0.98x0.95mm_HandSolder -> Resistor_SMD:R_0603_1608Metric_Pad0.98x0.95mm_HandSolder
- U1, U4, U6: value PDRV8243SDGQQ1 -> DRV8243HQDGQRQ1
- U12, U13: value ~ -> SI8640AB-B-IS1
- U15: value ~ -> 215079-4
- U3: footprint Library:SOT-583-8 -> Package_TO_SOT_SMD:SOT-583-8
- U5: footprint Library:SOT-23-5 -> Package_TO_SOT_SMD:SOT-23-5

Commit message: .
Parts:
- C1, C13, C14, C15, C17, C2, C21, C23, C26, C28, C29, C3, C4, C5: footprint Capacitor_SMD:C_0805_2012Metric_Pad1.18x1.45mm_HandSolder -> Library:C_0805_2012Metric_Pad1.18x1.45mm_HandSolder
- C10, C11, C12, C16, C18, C19, C20, C22, C24, C25, C27, C30, C31, C32, C33, C34, C35, C36, C37, C6, C7, C8, C9: footprint Capacitor_SMD:C_0603_1608Metric_Pad1.08x0.95mm_HandSolder -> Library:C_0603_1608Metric_Pad1.08x0.95mm_HandSolder
- D1: footprint LED_SMD:LED_0603_1608Metric_Pad1.05x0.95mm_HandSolder -> Library:LED_0603_1608Metric_Pad1.05x0.95mm_HandSolder
- J2, J7, J8, J9: footprint Connector_Wire:SolderWirePad_1x02_SMD_3x4mm -> Library:SolderWirePad_1x02_SMD_3x4mm
- J3: footprint Connector_PinHeader_2.54mm:PinHeader_1x04_P2.54mm_Vertical -> Library:PinHeader_1x04_P2.54mm_Vertical
- J4, J6: footprint Connector_PinHeader_2.54mm:PinHeader_1x03_P2.54mm_Vertical -> Library:PinHeader_1x03_P2.54mm_Vertical
- L1: footprint Inductor_SMD:SRP4021HMCT-1R5M_custom -> Library:SRP4021HMCT-1R5M_custom
- R1, R10, R11, R12, R13, R14, R15, R16, R17, R18, R19, R2, R20, R3, R4, R5, R6, R7, R8, R9: footprint Resistor_SMD:R_0603_1608Metric_Pad0.98x0.95mm_HandSolder -> Library:R_0603_1608Metric_Pad0.98x0.95mm_HandSolder
- U3: footprint Package_TO_SOT_SMD:SOT-583-8 -> Library:SOT-583-8
- U5: footprint Package_TO_SOT_SMD:SOT-23-5 -> Library:SOT-23-5
