File: electronics/picr_1_9tdi.kicad_pcb (KiCad board)
At the start: 4 copper layers, 50 x 50 mm, 92 parts, among them J1 10118193-0001LF, J2 Conn_01x02_Socket, J3 Conn_01x02_Socket, J3 Conn_01x03_Pin, J3 Conn_01x04_Socket, J4 Conn_01x03_Pin, J5 Conn_01x02_Socket, J6 Conn_01x03_Pin, J7 Conn_01x02_Socket, J8 Conn_01x02_Socket, J9 Conn_01x02_Socket, Q1 BUK6Y10-30PX, U1 DRV8243HQDGQRQ1, U10 215079-4, U11 215079-4, U12 SI8640AB-B-IS1, U13 SI8640AB-B-IS1, U14 MAX12930EASA+, U15 215079-4, U2 CM1223-02SO, U3 NCP718BSN500T1G, U3 TPS62933, U4 DRV8243HQDGQRQ1, U5 MIC5504-3.3YM5, U6 DRV8243HQDGQRQ1, U7 STM32G441KBT6, U8 20021121-00010T4LF, U9 215079-4

Commit message: .
Parts:
- C1, C13, C14, C15, C17, C2, C21, C23, C26, C28, C29, C3, C4, C5: footprint Library:C_0805_2012Metric_Pad1.18x1.45mm_HandSolder -> Capacitor_SMD:C_0805_2012Metric_Pad1.18x1.45mm_HandSolder
- C10, C11, C12, C16, C18, C19, C20, C22, C24, C25, C27, C30, C31, C32, C33, C34, C35, C36, C37, C6, C7, C8, C9: footprint Library:C_0603_1608Metric_Pad1.08x0.95mm_HandSolder -> Capacitor_SMD:C_0603_1608Metric_Pad1.08x0.95mm_HandSolder
- D1: footprint Library:LED_0603_1608Metric_Pad1.05x0.95mm_HandSolder -> LED_SMD:LED_0603_1608Metric_Pad1.05x0.95mm_HandSolder
- R1, R10, R11, R12, R13, R14, R15, R16, R17, R18, R19, R2, R20, R3, R4, R5, R6, R7, R8, R9: footprint Library:R_0603_1608Metric_Pad0.98x0.95mm_HandSolder -> Resistor_SMD:R_0603_1608Metric_Pad0.98x0.95mm_HandSolder

Commit message: .
Parts:
- C1, C13, C14, C15, C17, C2, C21, C23, C26, C28, C29, C3, C4, C5: footprint Capacitor_SMD:C_0805_2012Metric_Pad1.18x1.45mm_HandSolder -> Library:C_0805_2012Metric_Pad1.18x1.45mm_HandSolder
- C10, C11, C12, C16, C18, C19, C20, C22, C24, C25, C27, C30, C31, C32, C33, C34, C35, C36, C37, C6, C7, C8, C9: footprint Capacitor_SMD:C_0603_1608Metric_Pad1.08x0.95mm_HandSolder -> Library:C_0603_1608Metric_Pad1.08x0.95mm_HandSolder
- D1: footprint LED_SMD:LED_0603_1608Metric_Pad1.05x0.95mm_HandSolder -> Library:LED_0603_1608Metric_Pad1.05x0.95mm_HandSolder
- R1, R10, R11, R12, R13, R14, R15, R16, R17, R18, R19, R2, R20, R3, R4, R5, R6, R7, R8, R9: footprint Resistor_SMD:R_0603_1608Metric_Pad0.98x0.95mm_HandSolder -> Library:R_0603_1608Metric_Pad0.98x0.95mm_HandSolder

Commit message: .
Parts:
- removed the J3 at (203.8, 84.1)
- removed the J3 at (212.2, 66.0)
- added J3: Conn_01x04_Pin, Connector_PinHeader_2.54mm:PinHeader_1x04_P2.54mm_Vertical, F.Cu at (71.4, 69.5)
- added J5: Conn_01x02_Pin, Connector_PinHeader_2.54mm:PinHeader_1x02_P2.54mm_Vertical, F.Cu at (85.5, 60.5)
- C1, C13, C14, C15, C17, C2, C21, C23, C26, C28, C29, C3, C4, C5: footprint Library:C_0805_2012Metric_Pad1.18x1.45mm_HandSolder -> Capacitor_SMD:C_0805_2012Metric_Pad1.18x1.45mm_HandSolder
- C10, C11, C12, C16, C18, C19, C20, C22, C24, C25, C27, C30, C31, C32, C33, C34, C35, C36, C37, C6, C7, C8, C9: footprint Library:C_0603_1608Metric_Pad1.08x0.95mm_HandSolder -> Capacitor_SMD:C_0603_1608Metric_Pad1.08x0.95mm_HandSolder
- D1: footprint Library:LED_0603_1608Metric_Pad1.05x0.95mm_HandSolder -> LED_SMD:LED_0603_1608Metric_Pad1.05x0.95mm_HandSolder
- J4, J6: footprint Library:PinHeader_1x03_P2.54mm_Vertical -> Connector_PinHeader_2.54mm:PinHeader_1x03_P2.54mm_Vertical
- R1, R10, R11, R12, R13, R14, R15, R16, R17, R18, R19, R2, R20, R3, R4, R5, R6, R7, R8, R9: footprint Library:R_0603_1608Metric_Pad0.98x0.95mm_HandSolder -> Resistor_SMD:R_0603_1608Metric_Pad0.98x0.95mm_HandSolder
- moved C27 89.5 mm to (88.4, 75.0), turned to 180 degrees
- moved U8 41.4 mm to (114.0, 81.5), turned to 90 degrees
- moved U15 35.1 mm to (51.6, 78.3)
- moved C21 28.7 mm to (87.9, 79.3), turned to -90 degrees
- moved C25 25.3 mm to (103.6, 81.5), turned to 0 degrees
- moved R15 24.7 mm to (99.7, 88.2), turned to 90 degrees
- moved C22 16.7 mm to (103.7, 84.7), turned to 0 degrees
- moved U2 9.56 mm to (79.1, 81.5), turned to -90 degrees
- moved J1 8.90 mm to (69.5, 81.2)
- moved U14 0.94 mm to (93.7, 93.0)
- moved U6 0.28 mm to (106.2, 112.2)
- moved U13 0.23 mm to (107.6, 93.0)
- moved U4 0.09 mm to (92.8, 112.0)
Routing:
- net /PWM_TH_I: track 19.9 -> 0.00 mm, vias 2 -> 0
- net /PWM_M3_I: track 18.6 -> 0.00 mm, vias 2 -> 0
- net /PWM_M2_I: track 17.6 -> 0.00 mm, vias 2 -> 0
- net /M_NSLEEP_I: track 17.5 -> 0.00 mm, vias 2 -> 0
- net /M1_DIR_I: track 17.5 -> 0.00 mm, vias 2 -> 0
- net /M3_DIR_I: track 17.1 -> 0.00 mm, vias 2 -> 0
- net /PWM_M1_I: track 16.4 -> 0.00 mm
- net /M2_DIR_I: track 16.4 -> 0.00 mm
- net /PWM_GRB_I: track 6.17 -> 0.00 mm, vias 2 -> 0
- net /PWM_ANG_I: track 5.74 -> 0.00 mm
- net /VUSB: track 1.76 -> 0.00 mm
- net GND_MOT: track 0.77 -> 0.00 mm

Commit message: .
Parts:
- removed the C35 at (193.3, 65.4)
- removed the C36 at (193.3, 67.9)
- removed the C36 at (193.3, 70.4)
- removed the C5 at (206.6, 103.1)
- removed the C5 at (184.6, 65.4)
- removed the C9 at (79.4, 129.2)
- removed the J3 at (174.2, 66.3)
- removed the J5 at (174.2, 73.8)
- removed the R6 at (193.3, 88.0)
- removed the U3 at (221.2, 92.0)
- added C36: 0.1u, Capacitor_SMD:C_0603_1608Metric_Pad1.08x0.95mm_HandSolder, B.Cu at (96.5, 85.6)
- added C5: 10u, Capacitor_SMD:C_0805_2012Metric_Pad1.18x1.45mm_HandSolder, B.Cu at (85.3, 103.2)
- C1, C10, C11, C12, C13, C14, C15, C17, C19, C2, C20, C23, C26, C28, C29, C3, C30, C31, C37, C4, C6, C7, C8, C9, J2, L1, Q1, R13, R4, R7, R8, U14, U3, U8: moved to B.Cu
- U10, U11, U9: moved to F.Cu
- moved L1 139.0 mm to (85.4, 95.7)
- moved R19 128.6 mm to (75.9, 97.7), turned to 90 degrees
- moved R3 125.0 mm to (72.0, 110.8), turned to 180 degrees
- moved R2 121.5 mm to (75.4, 107.3), turned to 180 degrees
- moved C15 120.6 mm to (91.5, 109.7), turned to 90 degrees
- moved C13 117.4 mm to (95.5, 109.7), turned to 90 degrees
- moved C9 116.9 mm to (74.0, 110.7), turned to 90 degrees
- moved R11 115.7 mm to (88.4, 110.8), turned to 90 degrees
- moved R1 114.2 mm to (83.7, 107.3), turned to 180 degrees
- moved R4 113.5 mm to (90.2, 104.4), turned to -90 degrees
- moved C29 113.4 mm to (103.3, 109.9), turned to 90 degrees
- moved R12 113.2 mm to (84.7, 81.7), turned to 90 degrees
- moved R10 112.4 mm to (91.4, 107.0)
- moved R5 111.7 mm to (84.9, 109.8)
- moved C28 111.7 mm to (105.3, 109.9), turned to 90 degrees
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Connections:
- U14 pad 2: /PWM_GRB_I -> /PWM_ANG_I
- U14 pad 3: /PWM_ANG_I -> /PWM_GRB_I
- U14 pad 6: /PWM_ANG_O -> /PWM_GRB_O
- U14 pad 7: /PWM_GRB_O -> /PWM_ANG_O
- U5 pad 3: unconnected-(U5-EN-Pad3) -> /VUSB
Routing:
- net /M1_DIR_O: track 0.00 -> 1.31 mm
Other:
- outline, holes or cut-outs redrawn

Commit message: .
Routing:
- added copper zone on In1.Cu, net (none)
- added copper zone on In2.Cu, net (none)
Changed lines of the file:
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@@
 		(net 72)
+	)
+	(zone
+		(net 0)
+		(net_name "")
+		(layer "In1.Cu")
+		(hatch edge 0.5)
+		(connect_pads
+			(clearance 0.5)
+		)
+		(min_thickness 0.25)
+		(filled_areas_thickness no)
+		(fill yes
+			(thermal_gap 0.5)
+			(thermal_bridge_width 0.5)
+			(island_removal_mode 1)
+			(island_area_min 10)
+		)
+		(polygon
+			(pts
+				(xy 67.9 67.3) (xy 117.9 67.3) (xy 117.9 88.7) (xy 67.9 88.7)
+			)
+		)
+	)
+	(zone
+		(net 0)
+		(net_name "")
+		(layer "In1.Cu")
+		(hatch edge 0.5)
+		(connect_pads
+			(clearance 0.5)
+		)
+		(min_thickness 0.25)
+		(filled_areas_thickness no)
+		(fill yes
+			(thermal_gap 0.5)
+			(thermal_bridge_width 0.5)
+			(island_removal_mode 1)
+			(island_area_min 10)
+		)
+		(polygon
+			(pts
+				(xy 67.9 92.1) (xy 117.9 92.1) (xy 117.9 117.3) (xy 67.9 117.2)
+			)
+		)
+	)
+	(zone
+		(net 0)
+		(net_name "")
+		(layer "In2.Cu")
+		(hatch edge 0.5)
+		(priority 2)
+		(connect_pads
+			(clearance 0.5)
+		)
+		(min_thickness 0.25)
+		(filled_areas_thickness no)
+		(fill yes
+			(thermal_gap 0.5)
+			(thermal_bridge_width 0.5)
+			(island_removal_mode 1)
+			(island_area_min 10)
+		)
+		(polygon
+			(pts
+				(xy 67.9 92.1) (xy 67.9 117.2) (xy 117.9 117.3) (xy 117.9 92.1)
+			)
+		)
+	)
+	(zone
+		(net 0)
+		(net_name "")
+		(layer "In2.Cu")
+		(hatch edge 0.5)
+		(priority 1)
+		(connect_pads
+			(clearance 0.5)
+		)
+		(min_thickness 0.25)
+		(filled_areas_thickness no)
+		(fill yes
+			(thermal_gap 0.5)
+			(thermal_bridge_width 0.5)
+			(island_removal_mode 1)
+			(island_area_min 10)
+		)
+		(polygon
+			(pts
+				(xy 67.9 67.3) (xy 117.9 67.3) (xy 117.9 88.7) (xy 67.9 88.7)
+			)
+		)
 	)
 	(embedded_fonts no)

Commit message: .
Parts:
- moved J2 10.5 mm to (69.8, 105.1), turned to -90 degrees
- moved Q1 1.49 mm to (80.2, 103.6), turned to -90 degrees
- moved C33 1.22 mm to (84.7, 85.7), turned to 0 degrees
- moved C32 0.80 mm to (111.7, 85.7), turned to 0 degrees
- moved L1 0.61 mm to (85.5, 96.3)
- moved U8 0.30 mm to (71.7, 81.4)
- moved J1 0.20 mm to (69.5, 72.1)
- turned C20 to 90 degrees
- turned R15 to 180 degrees
Routing:
- added copper zone on B.Cu, net GND_MCU
- added copper zone on F.Cu, net GND_MCU
- added copper zone on B.Cu, net GND_MOT
- added copper zone on F.Cu, net GND_MOT
