File: electronics/picr_1_9tdi.kicad_pcb (KiCad board)
At the start: 4 copper layers, 50 x 50 mm, 84 parts, among them J1 10118193-0001LF, J2 Conn_01x02_Socket, J3 Conn_01x04_Pin, J4 Conn_01x03_Pin, J5 Conn_01x02_Pin, J6 Conn_01x03_Pin, J7 Conn_01x02_Socket, J8 Conn_01x02_Socket, J9 Conn_01x02_Socket, Q1 BUK6Y10-30PX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

Commit message: .
Routing:
- net /PWM_M2_O: track 31.6 -> 28.1 mm, vias 4 -> 2
- net GND_MOT: track 16.5 -> 13.6 mm, vias 142 -> 149
- net GND_MCU: track 23.0 -> 20.2 mm, vias 50 -> 53
- net /M1_DIR_O: track 39.3 -> 37.1 mm
- net /5V_MOT: track 79.5 -> 78.1 mm
- net /PWM_TH_O: track 7.80 -> 8.88 mm
- net /E_M1_B: track 10.1 -> 9.09 mm
- net +3.3V: track 127.6 -> 126.8 mm
- net /E_M1_A: track 13.4 -> 12.9 mm
- net /PWM_TH_I: track 16.6 -> 16.1 mm
- net /SWCLK: track 24.8 -> 24.3 mm

Commit message: .
Routing:
- net GND_MOT: track 13.6 -> 12.3 mm, vias 149 -> 150
- net GND_MCU: vias 53 -> 54

Commit message: .
Routing:
- net Net-(U1-SR): track 6.26 -> 3.38 mm
- net /PWM_ANG_O: track 26.8 -> 28.7 mm
- net /E_M2_B: track 19.0 -> 17.6 mm
- net /E_M2_A: track 15.1 -> 14.1 mm
- net /PWM_GRB_O: track 27.1 -> 27.8 mm
- net GND_MOT: track 12.3 -> 12.7 mm, vias 150 -> 159
- net GND_MCU: track 20.2 -> 20.5 mm, vias 54 -> 60
- net +3.3V: track 127.3 -> 127.4 mm, vias 5 -> 4
Other:
- board text added: "1.9 TDI"

Commit message: .
Routing:
- net GND_MCU: track 20.5 -> 19.5 mm, vias 60 -> 61

Commit message: .
Routing:
- net GND_MCU: vias 61 -> 62
